Commit message: fixed naming bug and added in robotiq

File: chonkur_manip_description/urdf/chonkur_macro.xacro (robot description, xacro)
@@ -105,4 +105,17 @@
       </gazebo>
     </xacro:if>
+    <xacro:property name="finger_type_prop" value="fngr_nail_v2" />
+    <xacro:include filename="$(find robotiq_hande_description)/urdf/robotiq_hande.xacro"/>
+    <xacro:robotiq_hande name="chonkur_hande" prefix="$(arg tf_prefix)" parent="$(arg tf_prefix)tool0" use_fake_hardware="$(arg use_fake_hardware)" com_port="/dev/ttyUSB0">
+      <origin xyz="0 0 0" rpy="0 0 0"/>
+    </xacro:robotiq_hande>
+    <!--If statements for the various types of gripper fingers-->
+    <xacro:if value="${finger_type_prop == 'fngr_nail_v2'}">
+      <xacro:include filename="$(find dextivr_hande_description)/urdf/hande_fingers_fngr_nail_v2.xacro"/>
+      <xacro:include filename="$(find dextivr_hande_description)/urdf/fngr_nail_v2_grasp_push_frames.xacro"/>
+    </xacro:if>
+    <!--Run the xacros from the files included above-->
+    <xacro:hande_fingers name="chonkur_hande_fingers" prefix="$(arg tf_prefix)"/>
+    <xacro:grasp_push_frames name="chonkur_grasp_push_frames" prefix="$(arg tf_prefix)"/>
   </xacro:macro>
 </robot>
