Commit message: created initial chonkur description

File: chonkur_manip_description/urdf/chonkur.urdf.xacro (robot description, xacro)
@@ -1,8 +1,15 @@
 <?xml version="1.0"?>
-<robot xmlns:xacro="http://wiki.ros.org/xacro" name="$(arg name)">
-  <xacro:arg name="name" default="chonkur"/>
+<robot xmlns:xacro="http://wiki.ros.org/xacro" name="chonkur">
+  <xacro:arg name="tf_prefix" default="" />
+  <xacro:arg name="use_fake_hardware" default="false" />
+  <xacro:arg name="headless_mode" default="false" />
   <xacro:arg name="ros2_control_name" default="chonkur"/>
-  <xacro:arg name="tf_prefix" default="" />
-  <xacro:arg name="headless_mode" default="false" />
-  <xacro:arg name="use_fake_hardware" default="false" />
   <xacro:include filename="$(find chonkur_manip_description)/urdf/chonkur_macro.xacro"/>
+  <link name="world" />
+  <xacro:chonkur
+    tf_prefix="$(arg tf_prefix)"
+    use_fake_hardware="$(arg use_fake_hardware)"
+    headless_mode="$(arg headless_mode)"
+    ros2_control_name="$(arg ros2_control_name)"
+    parent="world"/>
+</robot>

File: chonkur_manip_description/urdf/chonkur_macro.xacro (robot description, xacro)
@@ -9,6 +9,5 @@
     headless_mode:=false
     ros2_control_name:=chonkur
-    parent:=world
-  ">
+    parent:=world">
     <!-- parameters -->
     <xacro:arg name="joint_limit_params" default="$(find chonkur_manip_description)/config/joint_limits.yaml"/>
@@ -106,3 +105,4 @@
       </gazebo>
     </xacro:if>
+  </xacro:macro>
 </robot>

Commit message: got rid of args and fixed the default files

File: chonkur_manip_description/urdf/chonkur.urdf.xacro (robot description, xacro)
@@ -12,4 +12,6 @@
     headless_mode="$(arg headless_mode)"
     ros2_control_name="$(arg ros2_control_name)"
-    parent="world"/>
+    parent="world"
+    sim_gazebo="false"
+    sim_ignition="false"/>
 </robot>

File: chonkur_manip_description/urdf/chonkur_macro.xacro (robot description, xacro)
@@ -9,42 +9,9 @@
     headless_mode:=false
     ros2_control_name:=chonkur
-    parent:=world">
-    <!-- parameters -->
-    <xacro:arg name="joint_limit_params" default="$(find chonkur_manip_description)/config/ur10e/joint_limits.yaml"/>
-    <xacro:arg name="kinematics_params" default="$(find chonkur_manip_description)/config/ur10e/default_kinematics.yaml"/>
-    <xacro:arg name="physical_params" default="$(find chonkur_manip_description)/config/ur10e/physical_parameters.yaml"/>
-    <xacro:arg name="visual_params" default="$(find chonkur_manip_description)/config/ur10e/visual_parameters.yaml"/>
-    <xacro:arg name="transmission_hw_interface" default="hardware_interface/PositionJointInterface"/>
-    <xacro:arg name="safety_limits" default="false"/>
-    <xacro:arg name="safety_pos_margin" default="0.15"/>
-    <xacro:arg name="safety_k_position" default="20"/>
-    <!-- ros2_control related parameters -->
-    <xacro:arg name="headless_mode" default="false" />
-    <xacro:arg name="robot_ip" default="192.168.1.102" />
-    <xacro:arg name="script_filename" default="$(find ur_client_library)/resources/external_control.urscript"/>
-    <xacro:arg name="output_recipe_filename" default="$(find ur_robot_driver)/resources/rtde_output_recipe.txt"/>
-    <xacro:arg name="input_recipe_filename" default="$(find ur_robot_driver)/resources/rtde_input_recipe.txt"/>
-    <xacro:arg name="reverse_ip" default="0.0.0.0"/>
-    <xacro:arg name="script_command_port" default="50004"/>
-    <!--   tool communication related parameters-->
-    <xacro:arg name="use_tool_communication" default="false" />
-    <xacro:arg name="tool_voltage" default="0" />
-    <xacro:arg name="tool_parity" default="0" />
-    <xacro:arg name="tool_baud_rate" default="115200" />
-    <xacro:arg name="tool_stop_bits" default="1" />
-    <xacro:arg name="tool_rx_idle_chars" default="1.5" />
-    <xacro:arg name="tool_tx_idle_chars" default="3.5" />
-    <xacro:arg name="tool_device_name" default="/tmp/ttyUR" />
-    <xacro:arg name="tool_tcp_port" default="54321" />
-      <!-- Simulation parameters -->
-    <xacro:arg name="use_fake_hardware" default="false" />
-    <xacro:arg name="fake_sensor_commands" default="false" />
-    <xacro:arg name="sim_gazebo" default="false" />
-    <xacro:arg name="sim_ignition" default="false" />
-    <xacro:arg name="simulation_controllers" default="" />
-    <!-- initial position for simulations (Fake Hardware, Gazebo, Ignition) -->
-    <xacro:arg name="initial_positions_file" default="$(find chonkur_manip_description)/config/initial_positions.yaml"/>
+    parent:=world
+    sim_gazebo:=false
+    sim_ignition:=false">
     <!-- convert to property to use substitution in function -->
-    <xacro:property name="initial_positions_file" default="$(arg initial_positions_file)"/>
+    <xacro:property name="initial_positions_file" default="$(find chonkur_manip_description)/config/initial_positions.yaml"/>
     <!-- arm -->
     <xacro:ur_robot
@@ -52,37 +19,37 @@
       tf_prefix="${tf_prefix}"
       parent="${parent}"
-      joint_limits_parameters_file="$(arg joint_limit_params)"
-      kinematics_parameters_file="$(arg kinematics_params)"
-      physical_parameters_file="$(arg physical_params)"
-      visual_parameters_file="$(arg visual_params)"
-      transmission_hw_interface="$(arg transmission_hw_interface)"
-      safety_limits="$(arg safety_limits)"
-      safety_pos_margin="$(arg safety_pos_margin)"
-      safety_k_position="$(arg safety_k_position)"
-      use_fake_hardware="$(arg use_fake_hardware)"
-      fake_sensor_commands="$(arg fake_sensor_commands)"
-      sim_gazebo="$(arg sim_gazebo)"
-      sim_ignition="$(arg sim_ignition)"
-      headless_mode="$(arg headless_mode)"
+      joint_limits_parameters_file="$(find chonkur_manip_description)/config/joint_limits.yaml"
+      kinematics_parameters_file="$(find chonkur_manip_description)/config/calibrated_kinematics.yaml"
+      physical_parameters_file="$(find ur_description)/config/ur10e/physical_parameters.yaml"
+      visual_parameters_file="$(find ur_description)/config/ur10e/visual_parameters.yaml"
+      transmission_hw_interface="hardware_interface/PositionJointInterface"
+      safety_limits="false"
+      safety_pos_margin="0.15"
+      safety_k_position="20"
+      use_fake_hardware="${use_fake_hardware}"
+      fake_sensor_commands="false"
+      sim_gazebo="${sim_gazebo}"
+      sim_ignition="${sim_ignition}"
+      headless_mode="${headless_mode}"
       initial_positions="${xacro.load_yaml(initial_positions_file)}"
-      use_tool_communication="$(arg use_tool_communication)"
-      tool_voltage="$(arg tool_voltage)"
-      tool_parity="$(arg tool_parity)"
-      tool_baud_rate="$(arg tool_baud_rate)"
-      tool_stop_bits="$(arg tool_stop_bits)"
-      tool_rx_idle_chars="$(arg tool_rx_idle_chars)"
-      tool_tx_idle_chars="$(arg tool_tx_idle_chars)"
-      tool_device_name="$(arg tool_device_name)"
-      tool_tcp_port="$(arg tool_tcp_port)"
-      robot_ip="$(arg robot_ip)"
-      script_filename="$(arg script_filename)"
-      output_recipe_filename="$(arg output_recipe_filename)"
-      input_recipe_filename="$(arg input_recipe_filename)"
-      reverse_ip="$(arg reverse_ip)"
-      script_command_port="$(arg script_command_port)"
+      use_tool_communication="false"
+      tool_voltage="0"
+      tool_parity="0"
+      tool_baud_rate="115200"
+      tool_stop_bits="1"
+      tool_rx_idle_chars="1.5"
+      tool_tx_idle_chars="3.5"
+      tool_device_name="/tmp/ttyUR"
+      tool_tcp_port="54321"
+      robot_ip="192.168.1.102"
+      script_filename="$(find ur_client_library)/resources/external_control.urscript"
+      output_recipe_filename="$(find ur_robot_driver)/resources/rtde_output_recipe.txt"
+      input_recipe_filename="$(find ur_robot_driver)/resources/rtde_input_recipe.txt"
+      reverse_ip="0.0.0.0"
+      script_command_port="50004"
       >
       <origin xyz="0 0 0" rpy="0 0 0" />          <!-- position robot in the world -->
     </xacro:ur_robot>
-    <xacro:if value="$(arg sim_gazebo)">
+    <xacro:if value="${sim_gazebo}">
       <!-- Gazebo plugins -->
       <gazebo reference="world">
@@ -94,5 +61,5 @@
       </gazebo>
     </xacro:if>
-    <xacro:if value="$(arg sim_ignition)">
+    <xacro:if value="${sim_ignition}">
       <!-- Gazebo plugins -->
       <gazebo reference="world">
@@ -101,5 +68,5 @@
         <plugin filename="libign_ros2_control-system.so" name="ign_ros2_control::IgnitionROS2ControlPlugin">
           <parameters>$(arg simulation_controllers)</parameters>
-          <controller_manager_node_name>$(arg tf_prefix)controller_manager</controller_manager_node_name>
+          <controller_manager_node_name>${tf_prefix}controller_manager</controller_manager_node_name>
         </plugin>
       </gazebo>
@@ -107,5 +74,5 @@
     <xacro:property name="finger_type_prop" value="fngr_nail_v2" />
     <xacro:include filename="$(find robotiq_hande_description)/urdf/robotiq_hande.xacro"/>
-    <xacro:robotiq_hande name="chonkur_hande" prefix="$(arg tf_prefix)" parent="$(arg tf_prefix)tool0" use_fake_hardware="$(arg use_fake_hardware)" com_port="/dev/ttyUSB1">
+    <xacro:robotiq_hande name="chonkur_hande" prefix="${tf_prefix}" parent="${tf_prefix}tool0" use_fake_hardware="${use_fake_hardware}" com_port="/dev/ttyUSB1">
       <origin xyz="0 0 0" rpy="0 0 0"/>
     </xacro:robotiq_hande>
@@ -116,6 +83,6 @@
     </xacro:if>
     <!--Run the xacros from the files included above-->
-    <xacro:hande_fingers name="chonkur_hande_fingers" prefix="$(arg tf_prefix)"/>
-    <xacro:grasp_push_frames name="chonkur_grasp_push_frames" prefix="$(arg tf_prefix)"/>
+    <xacro:hande_fingers name="chonkur_hande_fingers" prefix="${tf_prefix}"/>
+    <xacro:grasp_push_frames name="chonkur_grasp_push_frames" prefix="${tf_prefix}"/>
   </xacro:macro>
 </robot>

Commit message: renamed package

File: chonkur_manip_description/urdf/chonkur.urdf.xacro (robot description, xacro)
@@ -5,5 +5,5 @@
   <xacro:arg name="headless_mode" default="false" />
   <xacro:arg name="ros2_control_name" default="chonkur"/>
-  <xacro:include filename="$(find chonkur_manip_description)/urdf/chonkur_macro.xacro"/>
+  <xacro:include filename="$(find chonkur_description)/urdf/chonkur_macro.xacro"/>
   <link name="world" />
   <xacro:chonkur

File: chonkur_manip_description/urdf/chonkur_macro.xacro (robot description, xacro)
@@ -15,5 +15,5 @@
     com_port_hande:=/dev/ttyUSB1">
     <!-- convert to property to use substitution in function -->
-    <xacro:property name="initial_positions_file" default="$(find chonkur_manip_description)/config/initial_positions.yaml"/>
+    <xacro:property name="initial_positions_file" default="$(find chonkur_description)/config/initial_positions.yaml"/>
     <!-- arm -->
     <xacro:ur_robot
@@ -21,6 +21,6 @@
       tf_prefix="${tf_prefix}"
       parent="${parent}"
-      joint_limits_parameters_file="$(find chonkur_manip_description)/config/joint_limits.yaml"
-      kinematics_parameters_file="$(find chonkur_manip_description)/config/calibrated_kinematics.yaml"
+      joint_limits_parameters_file="$(find chonkur_description)/config/joint_limits.yaml"
+      kinematics_parameters_file="$(find chonkur_description)/config/calibrated_kinematics.yaml"
       physical_parameters_file="$(find ur_description)/config/ur10e/physical_parameters.yaml"
       visual_parameters_file="$(find ur_description)/config/ur10e/visual_parameters.yaml"
