Commit message: modified moveit to allow for new clr package

File: clr_description/urdf/clr.urdf.xacro (robot description, xacro)
@@ -23,3 +23,10 @@
     ewellix_height_limit="0.53"
   />
+  <!-- creating world frame for moveit -->
+  <link name="world" />
+  <joint name="world_to_clr" type="fixed">
+    <parent link="world"/>
+    <child link="clr_base" />
+    <origin xyz="0 0 0" rpy="0 0 0"/>
+  </joint>
 </robot>

Commit message: updated entire urdf to match clr irl, macroized several links, view_robot.launch.py running

File: clr_description/urdf/clr.urdf.xacro (robot description, xacro)
@@ -5,5 +5,5 @@
   <xacro:arg name="headless_mode" default="false" />
   <xacro:include filename="$(find clr_description)/urdf/clr_macro.xacro"/>
-  <link name="clr_base" />
+  <link name="world" />
   <xacro:clr
     tf_prefix="$(arg tf_prefix)"
@@ -11,5 +11,5 @@
     headless_mode="$(arg headless_mode)"
     ros2_control_name="clr"
-    parent="clr_base"
+    parent="world"
     sim_gazebo="false"
     sim_ignition="false"
@@ -23,10 +23,3 @@
     ewellix_height_limit="0.53"
   />
-  <!-- creating world frame for moveit -->
-  <link name="world" />
-  <joint name="world_to_clr" type="fixed">
-    <parent link="world"/>
-    <child link="clr_base" />
-    <origin xyz="0 0 0" rpy="0 0 0"/>
-  </joint>
 </robot>

File: clr_description/urdf/clr_macro.xacro (robot description, xacro)
@@ -17,5 +17,20 @@
     ewellix_com_port:=/dev/ttyUSB0
     ewellix_height_limit:=0.53
+    ewellix_omit_plates:=true
   ">
+    <!-- CLR BASE JOINT -->
+    <joint name="${tf_prefix}clr_base_joint" type="fixed">
+      <parent link="${parent}"/>
+      <child link="${tf_prefix}clr_base"/>
+      <origin xyz="0 0 0" rpy="0 0 0"/>
+    </joint>
+    <!-- CLR BASE -->
+    <link name="${tf_prefix}clr_base">
+      <visual>
+        <geometry>
+          <mesh filename="file://$(find clr_description)/meshes/visual/clr_base.dae"/>
+        </geometry>
+      </visual>
+    </link>
     <!-- RAIL -->
     <xacro:include filename="$(find vention_rail_description)/urdf/vention_macro.urdf.xacro"/>
@@ -23,50 +38,70 @@
       name="${ros2_control_name}_rail"
       tf_prefix="${tf_prefix}"
+      parent="${tf_prefix}clr_base"
       use_fake_hardware="${use_fake_hardware}"
       ip_addr="${rail_ip}"
       port="${rail_port}"
       position_limit="${rail_position_limit}"
-      velocity_limit="${rail_velocity_limit}"/>
-    <!-- BASE JOINT OF CLR-->
-    <joint name="${tf_prefix}clr_base_joint" type="fixed">
-      <parent link="${tf_prefix}${parent}"/>
-      <child link="${tf_prefix}vention_rail_base_link" />
-      <origin xyz="0 0 0" rpy="0 0 0"/>
-    </joint>
-    <!-- EWELLIX 700 MM LIFT -->
+      velocity_limit="${rail_velocity_limit}"
+    >
+      <origin xyz="0.0874537 0.114017 0.300000"/>
+    </xacro:vention_rail>
+    <!-- CLR_CARRIAGE -->
+    <xacro:include filename="$(find clr_description)/urdf/clr_carriage.macro.xacro"/>
+    <xacro:clr_carriage
+      tf_prefix="${tf_prefix}"
+      parent="${tf_prefix}vention_rail_carriage"
+    >
+      <origin xyz="-0.003624 -0.0900 0.0185"/>
+    </xacro:clr_carriage>
+    <!-- LOWER_LIFT_PLATE -->
+    <xacro:include filename="$(find clr_description)/urdf/plates.macro.xacro"/>
+    <xacro:lower_lift_plate
+      tf_prefix="${tf_prefix}"
+      parent="${tf_prefix}clr_carriage"
+    >
+      <origin xyz="0 0 0.054525" rpy="0 0 0"/>
+    </xacro:lower_lift_plate>
+    <!-- LIFT -->
     <xacro:include filename="$(find ewellix_liftkit_description)/urdf/ewellix_lift.xacro"/>
     <xacro:ewellix_lift
       name="${ros2_control_name}_liftkit"
       tf_prefix="${tf_prefix}"
-      parent="${tf_prefix}vention_rail_carriage"
+      parent="${tf_prefix}lower_lift_plate"
       height_limit="${ewellix_height_limit}"
-      omit_plates="false"
+      omit_plates="${ewellix_omit_plates}}"
       use_fake_hardware="${use_fake_hardware}"
       com_port="${ewellix_com_port}"
-      />
-    <!-- parent joint does not exist for the lift so doing it here-->
-    <joint name="${tf_prefix}carriage_to_ewellix_lift_base_link" type="fixed">
-      <parent link="${tf_prefix}vention_rail_carriage"/>
-      <child link="${tf_prefix}ewellix_lift_base_link" />
-      <origin xyz="-0.1115 0.0 0.39" rpy="0 0 3.14159"/>
+    >
+      <origin xyz="0 0 0.249525" rpy="0 0 0"/>
+    </xacro:ewellix_lift>
+    <!-- UPPER_LIFT_PLATE -->
+    <xacro:upper_lift_plate
+      tf_prefix="$(arg tf_prefix)"
+      parent="$(arg tf_prefix)ewellix_lift_higher_link"
+    >
+      <origin xyz="0 0 0.253525" rpy="0 0 0"/>
+    </xacro:upper_lift_plate>
+    <!-- RIGHT_ANGLE_MOUNT -->
+    <xacro:include filename="$(find clr_description)/urdf/right_angle_mount.macro.xacro"/>
+    <xacro:right_angle_mount tf_prefix="$(arg tf_prefix)"/>
+    <!-- UPPER_LIFT_PLATE_TO_RIGHT_ANGLE_MOUNT -->
+    <joint name="upper_lift_plate_to_right_angle_mount" type="fixed">
+      <parent link="$(arg tf_prefix)upper_lift_plate"/>
+      <child link="$(arg tf_prefix)right_angle_mount"/>
+      <origin xyz="0 0 0.009525" rpy="0 0 0"/>
     </joint>
-    <!-- 90 degree mount-->
-    <link name="${tf_prefix}link_90deg">
-      <visual>
-        <geometry>
-          <mesh filename="file://$(find clr_description)/meshes/visual/clr_link_90deg_visual.dae"/>
-        </geometry>
-      </visual>
-    </link>
-    <joint name="${tf_prefix}base_to_90deg" type="fixed">
-      <parent link="${tf_prefix}ewellix_lift_top_link"/>
-      <child link="${tf_prefix}link_90deg" />
-      <origin xyz="0.0 0.0 0.0145" rpy="0 0 0"/>
-    </joint>
-    <link name="chonkur_mount_plate"/>
-    <joint name="${tf_prefix}chonkur_mount" type="fixed">
-      <parent link="${tf_prefix}link_90deg"/>
-      <child link="${tf_prefix}chonkur_mount_plate" />
-      <origin xyz="0 -0.136 0.1315"  rpy="-1.570796 3.14159 3.14159" />
+    <!-- UR10E_MOUNT_PLATE -->
+    <xacro:ur10e_mount_plate
+      tf_prefix="${tf_prefix}"
+      parent="${tf_prefix}right_angle_mount"
+    >
+      <origin xyz="0 0.112509 0.112509" rpy="0 0 0"/>
+    </xacro:ur10e_mount_plate>
+    <link name="${tf_prefix}ur10e_mount_link"/>
+    <joint name="chonkur_mount_joint" type="fixed">
+      <parent link="${tf_prefix}ur10e_mount_plate"/>
+      <child link="${tf_prefix}ur10e_mount_link"/>
+      <origin xyz="0 0.0225 0" rpy="${radians(-90)} 0 0"/>
     </joint>
     <!-- chonkur -->
@@ -77,5 +112,5 @@
       headless_mode="${headless_mode}"
       ros2_control_name="${ros2_control_name}_ur"
-      parent="chonkur_mount_plate"
+      parent="${tf_prefix}ur10e_mount_link"
       sim_gazebo="false"
       sim_ignition="false"
