Commit message: modified to have package:// instead of file://find

File: clr_description/urdf/clr_carriage.macro.xacro (robot description, xacro)
@@ -15,5 +15,5 @@
             <visual>
                 <geometry>
-                    <mesh filename= "file://$(find clr_description)/meshes/visual/clr_carriage.dae"/>
+                    <mesh filename= "package://clr_description/meshes/visual/clr_carriage.dae"/>
                 </geometry>
             </visual>

File: clr_description/urdf/plates.macro.xacro (robot description, xacro)
@@ -54,5 +54,5 @@
             <visual>
                 <geometry>
-                    <mesh filename= "file://$(find clr_description)/meshes/visual/ur10e_plate.dae"/>
+                    <mesh filename= "package://clr_description/meshes/visual/ur10e_plate.dae"/>
                 </geometry>
             </visual>

File: clr_description/urdf/right_angle_mount.macro.xacro (robot description, xacro)
@@ -6,5 +6,5 @@
             <visual>
                 <geometry>
-                    <mesh filename= "file://$(find clr_description)/meshes/visual/right_angle_mount.dae"/>
+                    <mesh filename= "package://clr_description/meshes/visual/right_angle_mount.dae"/>
                 </geometry>
             </visual>

Commit message: added collision for carriage coupler in clr_carriage macro

File: clr_description/urdf/clr_carriage.macro.xacro (robot description, xacro)
@@ -18,4 +18,22 @@
                 </geometry>
             </visual>
+            <collision>
+                <origin xyz="0 -0.0005 0.0225" rpy="0 0 0"/>
+                <geometry>
+                    <box size="0.403 0.404 0.045"/>
+                </geometry>
+            </collision>
+            <collision>
+                <origin xyz="-0.182 0.203 0.137" rpy="0 0 0"/>
+                <geometry>
+                    <box size="0.049 0.281 0.184"/>
+                </geometry>
+            </collision>
+            <collision>
+                <origin xyz="0.0220 0.276 0.157" rpy="0 0 0"/>
+                <geometry>
+                    <box size="0.359 0.135 0.0890"/>
+                </geometry>
+            </collision>
         </link>
     </xacro:macro>
