Commit message: added collisions to plate macros

File: clr_description/urdf/plates.macro.xacro (robot description, xacro)
@@ -19,4 +19,9 @@
                 </geometry>
             </visual>
+            <collision>
+                <geometry>
+                    <box size="0.310 0.310 0.01905"/>
+                </geometry>
+            </collision>
         </link>
     </xacro:macro>
@@ -38,4 +43,9 @@
                 </geometry>
             </visual>
+            <collision>
+                <geometry>
+                    <box size="0.225 0.225 0.01905"/>
+                </geometry>
+            </collision>
         </link>
     </xacro:macro>
@@ -57,4 +67,16 @@
                 </geometry>
             </visual>
+            <collision>
+                <origin xyz="0 0.005625 0" rpy="0 0 0"/>
+                <geometry>
+                    <box size="0.225 0.01125 0.225"/>
+                </geometry>
+            </collision>
+            <collision>
+                <origin xyz="0 0.016875 0" rpy="${radians(-90)} 0 0"/>
+                <geometry>
+                    <cylinder radius="0.095" length="0.01125"/>
+                </geometry>
+            </collision>
         </link>
     </xacro:macro>
