Commit message: Avoid error material 'aluminum' is not unique

File: clr_description/urdf/lift_camera.macro.xacro (robot description, xacro)
@@ -15,5 +15,5 @@
         <visual>
             <geometry>
-                <mesh filename= "package://clr_description/meshes/visual/lift_camera_mount.stl"/>
+                <mesh filename= "package://clr_description/meshes/visual/lift_camera_mount.stl" scale="0.001 0.001 0.001"/>
             </geometry>
         </visual>
@@ -26,11 +26,12 @@
     <!-- TODO Fix the origin -->
     <!-- Realsense camera -->
-    <!-- <xacro:include filename="$(find realsense2_description)/urdf/_d435.urdf.xacro"/>
-    <xacro:sensor_d435 parent="${tf_prefix}lift_camera_mount"
-                       use_nominal_extrinsics="true"
-                       use_mesh="true"
-                       name="lift_camera">
+    <xacro:property name="realsense_materials_defined" default="false" />
+    <xacro:unless value="${realsense_materials_defined}">
+        <xacro:property name="realsense_materials_defined" value="true" />
+    </xacro:unless>  <!--Avoid Error   material 'aluminum' is not unique.-->
+    <xacro:include filename="$(find realsense2_description)/urdf/_d435.urdf.xacro" ns="lift_camera_ns"/>
+    <xacro:lift_camera_ns.sensor_d435 parent="${tf_prefix}lift_camera_mount" use_nominal_extrinsics="true" use_mesh="true" name="lift_camera">
         <origin xyz="0.064 -0.006 -0.016" rpy="0 0 0"/>
-    </xacro:sensor_d435> -->
+    </xacro:lift_camera_ns.sensor_d435>
     </xacro:macro>
 </robot>

Commit message: only the one-line fix makes sense for non-unique material error

File: clr_description/urdf/lift_camera.macro.xacro (robot description, xacro)
@@ -26,8 +26,6 @@
     <!-- TODO Fix the origin -->
     <!-- Realsense camera -->
-    <xacro:property name="realsense_materials_defined" default="false" />
-    <xacro:unless value="${realsense_materials_defined}">
-        <xacro:property name="realsense_materials_defined" value="true" />
-    </xacro:unless>  <!--Avoid Error   material 'aluminum' is not unique.-->
+    <xacro:property name="realsense_materials_defined" default="true"/>
+     <!--Avoid Error   material 'aluminum' is not unique. (not sure why header guards in source code don't work)-->
     <xacro:include filename="$(find realsense2_description)/urdf/_d435.urdf.xacro" ns="lift_camera_ns"/>
     <xacro:lift_camera_ns.sensor_d435 parent="${tf_prefix}lift_camera_mount" use_nominal_extrinsics="true" use_mesh="true" name="lift_camera">

Commit message: realsense camera origin

File: clr_description/urdf/lift_camera.macro.xacro (robot description, xacro)
@@ -27,11 +27,9 @@
         </collision>
     </link>
-    <!-- TODO Fix the origin -->
     <!-- Realsense camera -->
-    <xacro:property name="realsense_materials_defined" default="true"/>
-     <!--Avoid Error   material 'aluminum' is not unique. (not sure why header guards in source code don't work)-->
+    <xacro:property name="realsense_materials_defined" default="true"/> <!--Avoid Error   material 'aluminum' is not unique. (not sure why header guards in source code don't work)-->
     <xacro:include filename="$(find realsense2_description)/urdf/_d435.urdf.xacro" ns="lift_camera_ns"/>
     <xacro:lift_camera_ns.sensor_d435 parent="${tf_prefix}lift_camera_mount" use_nominal_extrinsics="true" use_mesh="true" name="lift_camera">
-        <origin xyz="0.076 ${mount_width_meters} -0.185" rpy="0 0 0"/>
+        <origin xyz="0.076 0.01 -0.1725" rpy="3.1415 0 1.5708"/> <!--lift_camera_bottom_screw_frame-->
     </xacro:lift_camera_ns.sensor_d435>
     </xacro:macro>

Commit message: remove namespace + set realsense_materials_defined

File: clr_description/urdf/lift_camera.macro.xacro (robot description, xacro)
@@ -19,4 +19,5 @@
                 <mesh filename= "package://clr_description/meshes/visual/lift_camera_mount.stl"/>
             </geometry>
+            <color rgba="0.1 0.1 0.1 1"/>
         </visual>
         <collision>
@@ -28,9 +29,11 @@
     </link>
     <!-- Realsense camera -->
-    <xacro:property name="realsense_materials_defined" default="true"/> <!--Avoid Error   material 'aluminum' is not unique. (not sure why header guards in source code don't work)-->
-    <xacro:include filename="$(find realsense2_description)/urdf/_d435.urdf.xacro" ns="lift_camera_ns"/>
-    <xacro:lift_camera_ns.sensor_d435 parent="${tf_prefix}lift_camera_mount" use_nominal_extrinsics="true" use_mesh="true" name="lift_camera">
-        <origin xyz="0.076 0.01 -0.1725" rpy="3.1415 0 1.5708"/> <!--lift_camera_bottom_screw_frame-->
-    </xacro:lift_camera_ns.sensor_d435>
+    <xacro:property name="realsense_materials_defined" value="true" />
+    <!-- ^^ Avoid Error   material 'aluminum' is not unique. (not sure why header guards in source code don't work)-->
+    <!-- origin is lift_camera_bottom_screw_frame-->
+    <xacro:include filename="$(find realsense2_description)/urdf/_d435.urdf.xacro" />
+    <xacro:sensor_d435 parent="${tf_prefix}lift_camera_mount" use_nominal_extrinsics="true" use_mesh="true" name="lift_camera">
+        <origin xyz="0.076 0.01 -0.1725" rpy="3.1415 0 1.5708"/>
+    </xacro:sensor_d435>
     </xacro:macro>
 </robot>

Commit message: calibrated lift camera pose

File: clr_description/urdf/lift_camera.macro.xacro (robot description, xacro)
@@ -34,8 +34,13 @@
         Version 4.54.1 has header guards but they don't work as expected.
     -->
-    <!-- origin is lift_camera_bottom_screw_frame-->
+    <!-- Pose obtained from Measuring by hand. Origin is lift_camera_bottom_screw_frame-->
+    <!-- <xacro:include filename="$(find realsense2_description)/urdf/_d435.urdf.xacro" />
+    <xacro:sensor_d435 parent="${tf_prefix}lift_camera_mount" use_nominal_extrinsics="true" use_mesh="true" name="hand_measured_lift_camera">
+        <origin xyz="0.076 0.01 -0.1725" rpy="3.1415 0 1.5708"/>
+    </xacro:sensor_d435> -->
+    <!-- Pose after camera calibration -->
     <xacro:include filename="$(find realsense2_description)/urdf/_d435.urdf.xacro" />
-    <xacro:sensor_d435 parent="${tf_prefix}lift_camera_mount" use_nominal_extrinsics="true" use_mesh="true" name="lift_camera">
-        <origin xyz="0.076 0.01 -0.1725" rpy="3.1415 0 1.5708"/>
+    <xacro:sensor_d435 parent="${tf_prefix}lower_lift_plate" use_nominal_extrinsics="true" use_mesh="true" name="lift_camera">
+        <origin xyz="-0.007666 0.1069 0.3866" rpy="-3.0512 -0.0276 1.5884"/>
     </xacro:sensor_d435>
     </xacro:macro>
