Commit message: adjusted orientation of ur

File: clr_description/urdf/clr_macro.xacro (robot description, xacro)
@@ -103,5 +103,5 @@
       <parent link="${tf_prefix}ur10e_mount_plate"/>
       <child link="${tf_prefix}ur10e_mount_link"/>
-      <origin xyz="0 0.0225 0" rpy="${radians(-90)} 0 0"/>
+      <origin xyz="0 0.0225 0" rpy="${radians(-90)} ${radians(180)} 0"/>
     </joint>
     <!-- chonkur -->

Commit message: fixed bad ref in base mesh

File: clr_description/urdf/clr_macro.xacro (robot description, xacro)
@@ -29,5 +29,5 @@
       <visual>
         <geometry>
-          <mesh filename="file://$(find clr_description)/meshes/visual/clr_base.dae"/>
+          <mesh filename="package://clr_description/meshes/visual/clr_base.dae"/>
         </geometry>
       </visual>

Commit message: added collision objects to clr_base link

File: clr_description/urdf/clr_macro.xacro (robot description, xacro)
@@ -32,4 +32,52 @@
         </geometry>
       </visual>
+      <collision>
+        <origin xyz="0 0 0.15" rpy="0 0 0"/>
+        <geometry>
+          <box size="2.43 0.81 0.30"/>
+        </geometry>
+      </collision>
+      <collision>
+        <origin xyz="0 0.315007 0.354694" rpy="0 0 0"/>
+        <geometry>
+          <box size="2.11500 0.179992 0.109387"/>
+        </geometry>
+      </collision>
+      <collision>
+        <origin xyz="0 -0.314989 0.592500" rpy="0 0 0"/>
+        <geometry>
+          <box size="1.88999 0.179978 0.585000"/>
+        </geometry>
+      </collision>
+      <collision>
+        <origin xyz="0.440106 0.495008 0.150000" rpy="0 0 0"/>
+        <geometry>
+          <box size="0.0899922 0.180010 0.300000"/>
+        </geometry>
+      </collision>
+      <collision>
+        <origin xyz="-0.446456 0.495008 0.150000" rpy="0 0 0"/>
+        <geometry>
+          <box size="0.0899922 0.180010 0.300000"/>
+        </geometry>
+      </collision>
+      <collision>
+        <origin xyz="0 -0.504978 0.442500" rpy="0 0 0"/>
+        <geometry>
+          <box size="1.88999 0.200000 0.885000"/>
+        </geometry>
+      </collision>
+      <collision>
+        <origin xyz="-1.17000 0 0.310844" rpy="0 0 0"/>
+        <geometry>
+          <box size="0.0899922 0.0899922 0.0216890"/>
+        </geometry>
+      </collision>
+      <collision>
+        <origin xyz="1.17000 0 0.310844" rpy="0 0 0"/>
+        <geometry>
+          <box size="0.0899922 0.0899922 0.0216890"/>
+        </geometry>
+      </collision>
     </link>
     <!-- RAIL -->

Commit message: updated lift macro origin to reflect increased lower_link height change in ewellix_lift_kit branch of same name

File: clr_description/urdf/clr_macro.xacro (robot description, xacro)
@@ -122,5 +122,5 @@
       com_port="${ewellix_com_port}"
     >
-      <origin xyz="0 0 0.249525" rpy="0 0 0"/>
+      <origin xyz="0 0 0.295" rpy="0 0 0"/>
     </xacro:ewellix_lift>
     <!-- UPPER_LIFT_PLATE -->

Commit message: added safety lights

File: clr_description/urdf/clr_macro.xacro (robot description, xacro)
@@ -105,4 +105,44 @@
       <origin xyz="-0.003624 -0.0900 0.0185"/>
     </xacro:clr_carriage>
+    <!-- SAFETY_LIGHTS -->
+    <material name="safety_light_blue">
+      <color rgba="0 0 0.5 0.8"/>
+    </material>
+    <link name="${tf_prefix}motor_side_estop_light">
+      <visual>
+        <geometry>
+          <box size="0.05 0.05 0.381"/>
+        </geometry>
+        <!-- <material name="safety_light_blue" />         -->
+      </visual>
+      <collision>
+        <geometry>
+          <box size="0.05 0.05 0.381"/>
+        </geometry>
+      </collision>
+    </link>
+    <joint name="${tf_prefix}motor_side_estop_light_joint" type="fixed">
+      <parent link="${tf_prefix}clr_carriage"/>
+      <child link="${tf_prefix}motor_side_estop_light"/>
+      <origin xyz="-0.0395 -0.296 0.5" rpy="0 0 0"/>
+    </joint>
+    <link name="${tf_prefix}end_estop_light">
+      <visual>
+        <geometry>
+          <box size="0.05 0.05 0.381"/>
+        </geometry>
+        <!-- <material name="safety_light_blue" />         -->
+      </visual>
+      <collision>
+        <geometry>
+          <box size="0.05 0.05 0.381"/>
+        </geometry>
+      </collision>
+    </link>
+    <joint name="${tf_prefix}end_estop_light_joint" type="fixed">
+      <parent link="${tf_prefix}clr_carriage"/>
+      <child link="${tf_prefix}end_estop_light"/>
+      <origin xyz="1.815 -0.296 0.3" rpy="0 0 0"/>
+    </joint>
     <!-- LOWER_LIFT_PLATE -->
     <xacro:include filename="$(find clr_description)/urdf/plates.macro.xacro"/>

Commit message: making estop lights w.r.t. clr_base instead of carriage

File: clr_description/urdf/clr_macro.xacro (robot description, xacro)
@@ -123,7 +123,7 @@
     </link>
     <joint name="${tf_prefix}motor_side_estop_light_joint" type="fixed">
-      <parent link="${tf_prefix}clr_carriage"/>
+      <parent link="${tf_prefix}clr_base"/>
       <child link="${tf_prefix}motor_side_estop_light"/>
-      <origin xyz="-0.0395 -0.296 0.5" rpy="0 0 0"/>
+      <origin xyz="-0.925 -0.272 0.914" rpy="0 0 0"/>
     </joint>
     <link name="${tf_prefix}end_estop_light">
@@ -141,7 +141,7 @@
     </link>
     <joint name="${tf_prefix}end_estop_light_joint" type="fixed">
-      <parent link="${tf_prefix}clr_carriage"/>
+      <parent link="${tf_prefix}clr_base"/>
       <child link="${tf_prefix}end_estop_light"/>
-      <origin xyz="1.815 -0.296 0.3" rpy="0 0 0"/>
+      <origin xyz="0.929 -0.272 0.714" rpy="0 0 0"/>
     </joint>
     <!-- LOWER_LIFT_PLATE -->

Commit message: camera added to clr_macro.xacro

File: clr_description/urdf/clr_macro.xacro (robot description, xacro)
@@ -166,4 +166,13 @@
       <origin xyz="0 0 0.295" rpy="0 0 0"/>
     </xacro:ewellix_lift>
+    <!-- LIFT CAMERA + MOUNT -->
+    <!-- TODO: FIX ORIGIN -->
+    <xacro include filename="$(find clr_description)/urdf/lift_camera.macro.xacro"/>
+    <xacro:lift_camera
+      tf_prefix="${tf_prefix}"
+      parent="${tf_prefix}ewellix_lift_lower_link"
+    >
+      <origin xyz="0 0 0" rpy="0 0 0"/>
+    </xacro:lift_camera>
     <!-- UPPER_LIFT_PLATE -->
     <xacro:upper_lift_plate

File: clr_description/urdf/lift_camera.macro.xacro (robot description, xacro)
@@ -2,6 +2,6 @@
 <robot xmlns:xacro="http://www.ros.org/wiki/xacro">
     <xacro:macro name="lift_camera" params="
-        tf_prefix
-        parent
+        tf_prefix:=''
+        parent:=world
         *origin
     ">

Commit message: added lift_camera_mount (still wip)

File: clr_description/urdf/clr_macro.xacro (robot description, xacro)
@@ -168,5 +168,5 @@
     <!-- LIFT CAMERA + MOUNT -->
     <!-- TODO: FIX ORIGIN -->
-    <xacro include filename="$(find clr_description)/urdf/lift_camera.macro.xacro"/>
+    <xacro:include filename="$(find clr_description)/urdf/lift_camera.macro.xacro"/>
     <xacro:lift_camera
       tf_prefix="${tf_prefix}"

File: clr_description/urdf/lift_camera.macro.xacro (robot description, xacro)
@@ -6,5 +6,5 @@
         *origin
     ">
-    <joint name="${tf_prefix}lift_camera_base_joint" type="fixed">
+    <joint name="${tf_prefix}lift_camera_mount_base_joint" type="fixed">
         <parent link="${parent}"/>
         <child link="${tf_prefix}lift_camera_mount"/>
@@ -15,10 +15,10 @@
         <visual>
             <geometry>
-                <!-- <mesh filename= "package://chonkur_description/meshes/visual/ur_realsense_short_mount_tube.stl"/> -->
+                <mesh filename= "package://clr_description/meshes/visual/lift_camera_mount.stl"/>
             </geometry>
         </visual>
         <collision>
             <geometry>
-                <!-- <mesh filename= "package://chonkur_description/meshes/visual/ur_realsense_short_mount_tube.stl"/> -->
+                <box size="0.145 0.15 0.01135"/> <!--meters -->
             </geometry>
         </collision>
@@ -31,5 +31,5 @@
                        use_mesh="true"
                        name="lift_camera">
-        <origin xyz="-0.064 -0.003 0.016" rpy="0.136 -1.429 -0.128"/>
+        <origin xyz="0.064 -0.006 -0.016" rpy="0 0 0"/>
     </xacro:sensor_d435>
     </xacro:macro>

Commit message: lift_camera_mount urdf

File: clr_description/urdf/clr_macro.xacro (robot description, xacro)
@@ -167,5 +167,4 @@
     </xacro:ewellix_lift>
     <!-- LIFT CAMERA + MOUNT -->
-    <!-- TODO FIX ORIGIN -->
     <xacro:include filename="$(find clr_description)/urdf/lift_camera.macro.xacro"/>
     <xacro:lift_camera
@@ -173,5 +172,5 @@
       parent="${tf_prefix}ewellix_lift_lower_link"
     >
-      <origin xyz="0 0 0" rpy="0 0 0"/>
+      <origin xyz="-0.0772 0.08785 0.2635" rpy="0 0 0"/>
     </xacro:lift_camera>
     <!-- UPPER_LIFT_PLATE -->

File: clr_description/urdf/lift_camera.macro.xacro (robot description, xacro)
@@ -4,4 +4,7 @@
         tf_prefix:=''
         parent:=world
+        mount_width_meters:=0.14
+        mount_height_meters:=0.2
+        mount_depth_meters:=0.01135
         *origin
     ">
@@ -11,14 +14,14 @@
         <xacro:insert_block name="origin"/>
     </joint>
-    <!-- TODO Get mesh of mount, as well as mesh of the cable management block that mounts on -->
     <link name="${tf_prefix}lift_camera_mount">
         <visual>
             <geometry>
-                <mesh filename= "package://clr_description/meshes/visual/lift_camera_mount.stl" scale="0.001 0.001 0.001"/>
+                <mesh filename= "package://clr_description/meshes/visual/lift_camera_mount.stl"/>
             </geometry>
         </visual>
         <collision>
+            <origin rpy="0 0 0" xyz="${mount_width_meters/2} ${-1*mount_depth_meters/2} ${-1*mount_height_meters/2}"/>
             <geometry>
-                <box size="0.145 0.15 0.01135"/> <!--meters -->
+                <box size="${mount_width_meters} ${mount_depth_meters} ${mount_height_meters}"/> <!--meters -->
             </geometry>
         </collision>
@@ -30,5 +33,5 @@
     <xacro:include filename="$(find realsense2_description)/urdf/_d435.urdf.xacro" ns="lift_camera_ns"/>
     <xacro:lift_camera_ns.sensor_d435 parent="${tf_prefix}lift_camera_mount" use_nominal_extrinsics="true" use_mesh="true" name="lift_camera">
-        <origin xyz="0.064 -0.006 -0.016" rpy="0 0 0"/>
+        <origin xyz="0.076 ${mount_width_meters} -0.185" rpy="0 0 0"/>
     </xacro:lift_camera_ns.sensor_d435>
     </xacro:macro>

Commit message: tweaked mount position so it is not intersecting lower lift

File: clr_description/urdf/clr_macro.xacro (robot description, xacro)
@@ -174,5 +174,5 @@
       parent="${tf_prefix}ewellix_lift_lower_link"
     >
-      <origin xyz="-0.0772 0.08785 0.2635" rpy="0 0 0"/>
+      <origin xyz="-0.0772 0.095 0.2635" rpy="0 0 0"/>
     </xacro:lift_camera>
     <!-- UPPER_LIFT_PLATE -->

Commit message: Fix prefix arg formatting

File: clr_description/urdf/clr_macro.xacro (robot description, xacro)
@@ -186,6 +186,6 @@
     <!-- UPPER_LIFT_PLATE -->
     <xacro:upper_lift_plate
-      tf_prefix="$(arg tf_prefix)"
-      parent="$(arg tf_prefix)ewellix_lift_higher_link"
+      tf_prefix="${tf_prefix}"
+      parent="${tf_prefix}ewellix_lift_higher_link"
     >
       <origin xyz="0 0 0.253525" rpy="0 0 0"/>
@@ -193,9 +193,9 @@
     <!-- RIGHT_ANGLE_MOUNT -->
     <xacro:include filename="$(find clr_description)/urdf/right_angle_mount.macro.xacro"/>
-    <xacro:right_angle_mount tf_prefix="$(arg tf_prefix)"/>
+    <xacro:right_angle_mount tf_prefix="${tf_prefix}"/>
     <!-- UPPER_LIFT_PLATE_TO_RIGHT_ANGLE_MOUNT -->
     <joint name="upper_lift_plate_to_right_angle_mount" type="fixed">
-      <parent link="$(arg tf_prefix)upper_lift_plate"/>
-      <child link="$(arg tf_prefix)right_angle_mount"/>
+      <parent link="${tf_prefix}upper_lift_plate"/>
+      <child link="${tf_prefix}right_angle_mount"/>
       <origin xyz="0 0 0.009525" rpy="0 0 0"/>
     </joint>

Commit message: Add dual clr config and update prefixes

File: clr_description/urdf/clr_macro.xacro (robot description, xacro)
@@ -112,5 +112,5 @@
     </xacro:clr_carriage>
     <!-- SAFETY_LIGHTS -->
-    <material name="safety_light_blue">
+    <material name="${tf_prefix}safety_light_blue">
       <color rgba="0 0 0.5 0.8"/>
     </material>
@@ -120,5 +120,5 @@
           <box size="0.05 0.05 0.381"/>
         </geometry>
-        <material name="safety_light_blue" />
+        <material name="${tf_prefix}safety_light_blue" />
       </visual>
       <collision>
@@ -138,5 +138,5 @@
           <box size="0.05 0.05 0.381"/>
         </geometry>
-        <material name="safety_light_blue" />
+        <material name="${tf_prefix}safety_light_blue" />
       </visual>
       <collision>
@@ -195,5 +195,5 @@
     <xacro:right_angle_mount tf_prefix="${tf_prefix}"/>
     <!-- UPPER_LIFT_PLATE_TO_RIGHT_ANGLE_MOUNT -->
-    <joint name="upper_lift_plate_to_right_angle_mount" type="fixed">
+    <joint name="${tf_prefix}upper_lift_plate_to_right_angle_mount" type="fixed">
       <parent link="${tf_prefix}upper_lift_plate"/>
       <child link="${tf_prefix}right_angle_mount"/>
@@ -208,5 +208,5 @@
     </xacro:ur10e_mount_plate>
     <link name="${tf_prefix}ur10e_mount_link"/>
-    <joint name="chonkur_mount_joint" type="fixed">
+    <joint name="${tf_prefix}chonkur_mount_joint" type="fixed">
       <parent link="${tf_prefix}ur10e_mount_plate"/>
       <child link="${tf_prefix}ur10e_mount_link"/>
