Commit message: adding ewellix hw calibration file

File: clr_description/urdf/clr_macro.xacro (robot description, xacro)
@@ -161,4 +161,5 @@
     <!-- LIFT -->
     <xacro:include filename="$(find ewellix_liftkit_description)/urdf/ewellix_lift.xacro"/>
+    <xacro:property name="ewellix_hw_calibration_file" value="$(find clr_description)/config/clr_ewellix_config.yaml"/>
     <xacro:ewellix_lift
       name="${ros2_control_name}_liftkit"
@@ -171,4 +172,5 @@
       is_700="true"
       is_500="false"
+      hw_calibration="${xacro.load_yaml(ewellix_hw_calibration_file)}"
       generate_ros2_control_tag="${generate_ros2_control_tag}"
     >

Commit message: removed motor side safety light from urdf

File: clr_description/urdf/clr_macro.xacro (robot description, xacro)
@@ -115,22 +115,4 @@
       <color rgba="0 0 0.5 0.8"/>
     </material>
-    <link name="${tf_prefix}motor_side_estop_light">
-      <visual>
-        <geometry>
-          <box size="0.05 0.05 0.381"/>
-        </geometry>
-        <material name="${tf_prefix}safety_light_blue" />
-      </visual>
-      <collision>
-        <geometry>
-          <box size="0.05 0.05 0.381"/>
-        </geometry>
-      </collision>
-    </link>
-    <joint name="${tf_prefix}motor_side_estop_light_joint" type="fixed">
-      <parent link="${tf_prefix}clr_base"/>
-      <child link="${tf_prefix}motor_side_estop_light"/>
-      <origin xyz="-0.925 -0.272 0.914" rpy="0 0 0"/>
-    </joint>
     <link name="${tf_prefix}end_estop_light">
       <visual>
