Commit message: no slashes in joint names...

File: clr_description/urdf/dualing_clrs.urdf.xacro (robot description, xacro)
@@ -9,8 +9,8 @@
       <parent link="world"/>
       <child link="world_to_left_link"/>
-    <origin xyz="0 0.75 0" rpy="0 0 0"/>
+    <origin xyz="0 1.0 0" rpy="0 0 3.14159"/>
   </joint>
   <xacro:clr
-    tf_prefix="left/"
+    tf_prefix="left_"
     parent="world_to_left_link"
     use_fake_hardware="true"
@@ -21,8 +21,8 @@
     <parent link="world"/>
     <child link="world_to_right_link"/>
-    <origin xyz="0 -0.75 0" rpy="0 0 0"/>
+    <origin xyz="0 -1.0 0" rpy="0 0 0"/>
   </joint>
   <xacro:clr
-    tf_prefix="right/"
+    tf_prefix="right_"
     parent="world_to_right_link"
     use_fake_hardware="true"
