Commit message: added end effector stack macro and meshes

File: chonkur_description/urdf/chonkur_macro.xacro (robot description, xacro)
@@ -74,8 +74,15 @@
       </gazebo>
     </xacro:if>
+    <!-- END EFFECTOR STACK -->
+    <xacro:include filename="$(find chonkur_description)/urdf/endeff_stack_macro.xacro"/>
+    <xacro:endeff_stack
+      tf_prefix="${tf_prefix}"
+      parent="${tf_prefix}tool0">
+      <origin xyz="0 0 0" rpy="0 0 0"/>
+    </xacro:endeff_stack>
     <xacro:property name="finger_type_prop" value="fngr_nail_v2" />
     <xacro:include filename="$(find robotiq_hande_description)/urdf/robotiq_hande.xacro"/>
-    <xacro:robotiq_hande name="chonkur_hande" prefix="${tf_prefix}" parent="${tf_prefix}tool0" use_fake_hardware="${use_fake_hardware}" com_port="${com_port_hande}">
-      <origin xyz="0 0 0" rpy="0 0 0"/>
+    <xacro:robotiq_hande name="chonkur_hande" prefix="${tf_prefix}" parent="${tf_prefix}robotiq_hand-e_adapter_old" use_fake_hardware="${use_fake_hardware}" com_port="${com_port_hande}">
+      <origin xyz="0 0 0.014" rpy="0 0 ${radians(-90)}"/>
     </xacro:robotiq_hande>
     <!--If statements for the various types of gripper fingers-->

Commit message: updated hand-e macro origin

File: chonkur_description/urdf/chonkur_macro.xacro (robot description, xacro)
@@ -84,5 +84,5 @@
     <xacro:include filename="$(find robotiq_hande_description)/urdf/robotiq_hande.xacro"/>
     <xacro:robotiq_hande name="chonkur_hande" prefix="${tf_prefix}" parent="${tf_prefix}robotiq_hand-e_adapter_old" use_fake_hardware="${use_fake_hardware}" com_port="${com_port_hande}">
-      <origin xyz="0 0 0.014" rpy="0 0 ${radians(-90)}"/>
+      <origin xyz="0 0 0.011" rpy="0 0 ${radians(-90)}"/>
     </xacro:robotiq_hande>
     <!--If statements for the various types of gripper fingers-->

Commit message: updating eef stackup to be in the correct orientation

File: chonkur_description/urdf/chonkur_macro.xacro (robot description, xacro)
@@ -79,5 +79,5 @@
       tf_prefix="${tf_prefix}"
       parent="${tf_prefix}tool0">
-      <origin xyz="0 0 0" rpy="0 0 0"/>
+      <origin xyz="0 0 0" rpy="0 0 ${radians(90)}"/>
     </xacro:endeff_stack>
     <xacro:property name="finger_type_prop" value="fngr_nail_v2" />

Commit message: added a temp frame for moveit studio purposes

File: chonkur_description/urdf/chonkur_macro.xacro (robot description, xacro)
@@ -94,4 +94,10 @@
     <xacro:hande_fingers name="chonkur_hande_fingers" prefix="${tf_prefix}"/>
     <xacro:grasp_push_frames name="chonkur_grasp_push_frames" prefix="${tf_prefix}"/>
+    <link name="manual_grasp_link" />
+    <joint name="${tf_prefix}temp_studio_joint" type="fixed">
+      <parent link="${tf_prefix}grasp_frame"/>
+      <child link="${tf_prefix}manual_grasp_link"/>
+      <origin xyz="0 0 0" rpy="0 0 0"/>
+    </joint>
   </xacro:macro>
 </robot>

Commit message: flipped manual_grasp_link about z by 180deg

File: chonkur_description/urdf/chonkur_macro.xacro (robot description, xacro)
@@ -98,5 +98,5 @@
       <parent link="${tf_prefix}grasp_frame"/>
       <child link="${tf_prefix}manual_grasp_link"/>
-      <origin xyz="0 0 0" rpy="0 0 0"/>
+      <origin xyz="0 0 0" rpy="0 0 ${radians(180)}"/>
     </joint>
   </xacro:macro>

Commit message: changed finger macro call to v2_m

File: chonkur_description/urdf/chonkur_macro.xacro (robot description, xacro)
@@ -82,4 +82,5 @@
     </xacro:endeff_stack>
     <xacro:property name="finger_type_prop" value="fngr_nail_v2" />
+    <xacro:property name="finger_type_prop" value="fngr_v2_m" />
     <xacro:include filename="$(find robotiq_hande_description)/urdf/robotiq_hande.xacro"/>
     <xacro:robotiq_hande name="chonkur_hande" prefix="${tf_prefix}" parent="${tf_prefix}robotiq_hand-e_adapter_old" use_fake_hardware="${use_fake_hardware}" com_port="${com_port_hande}">
@@ -90,4 +91,8 @@
       <xacro:include filename="$(find dextivr_hande_description)/urdf/hande_fingers_fngr_nail_v2.xacro"/>
       <xacro:include filename="$(find dextivr_hande_description)/urdf/fngr_nail_v2_grasp_push_frames.xacro"/>
+    </xacro:if>
+    <xacro:if value="${finger_type_prop == 'fngr_v2_m'}">
+      <xacro:include filename="$(find dextivr_hande_description)/urdf/hande_fingers_v2_m.xacro"/>
+      <xacro:include filename="$(find dextivr_hande_description)/urdf/fngr_v2_m_grasp_push_frames.xacro"/>
     </xacro:if>
     <!--Run the xacros from the files included above-->

Commit message: Moving the adapter plate into the robotiq hande repo.

File: chonkur_description/urdf/chonkur_macro.xacro (robot description, xacro)
@@ -81,9 +81,8 @@
       <origin xyz="0 0 0" rpy="0 0 ${radians(90)}"/>
     </xacro:endeff_stack>
-    <xacro:property name="finger_type_prop" value="fngr_nail_v2" />
     <xacro:property name="finger_type_prop" value="fngr_v2_m" />
     <xacro:include filename="$(find robotiq_hande_description)/urdf/robotiq_hande.xacro"/>
-    <xacro:robotiq_hande name="chonkur_hande" prefix="${tf_prefix}" parent="${tf_prefix}robotiq_hand-e_adapter_old" use_fake_hardware="${use_fake_hardware}" com_port="${com_port_hande}">
-      <origin xyz="0 0 0.011" rpy="0 0 ${radians(-90)}"/>
+    <xacro:robotiq_hande name="chonkur_hande" tf_prefix="${tf_prefix}" parent="${tf_prefix}ur_realsense_mount" use_fake_hardware="${use_fake_hardware}" com_port="${com_port_hande}">
+      <origin xyz="0 0 0.003" rpy="0 0 ${radians(-90)}"/>
     </xacro:robotiq_hande>
     <!--If statements for the various types of gripper fingers-->
@@ -97,6 +96,6 @@
     </xacro:if>
     <!--Run the xacros from the files included above-->
-    <xacro:hande_fingers name="chonkur_hande_fingers" prefix="${tf_prefix}"/>
-    <xacro:grasp_push_frames name="chonkur_grasp_push_frames" prefix="${tf_prefix}"/>
+    <xacro:hande_fingers name="chonkur_hande_fingers" tf_prefix="${tf_prefix}"/>
+    <xacro:grasp_push_frames name="chonkur_grasp_push_frames" tf_prefix="${tf_prefix}"/>
     <link name="manual_grasp_link" />
     <joint name="${tf_prefix}temp_studio_joint" type="fixed">

File: chonkur_description/urdf/endeff_stack_macro.xacro (robot description, xacro)
@@ -47,16 +47,4 @@
         <origin xyz="-0.065 -0.006 0.010" rpy="0.048 -1.392 -0.047"/>
     </xacro:sensor_d435>
-    <joint name="${tf_prefix}realsense_mount_to_hand-e_adapter" type="fixed">
-        <parent link="${tf_prefix}ur_realsense_mount"/>
-        <child link="${tf_prefix}robotiq_hand-e_adapter_old"/>
-        <origin xyz="0 0 0.003" rpy="0 0 0"/>
-    </joint>
-    <link name="${tf_prefix}robotiq_hand-e_adapter_old">
-        <visual>
-            <geometry>
-                <mesh filename= "package://chonkur_description/meshes/visual/robotiq_hand-e_adapter_old.dae"/>
-            </geometry>
-        </visual>
-    </link>
     </xacro:macro>
 </robot>

Commit message: Updating robotiq adapter plate transform.

File: chonkur_description/urdf/chonkur_macro.xacro (robot description, xacro)
@@ -84,5 +84,5 @@
     <xacro:include filename="$(find robotiq_hande_description)/urdf/robotiq_hande.xacro"/>
     <xacro:robotiq_hande name="chonkur_hande" tf_prefix="${tf_prefix}" parent="${tf_prefix}ur_realsense_mount" use_fake_hardware="${use_fake_hardware}" com_port="${com_port_hande}">
-      <origin xyz="0 0 0.003" rpy="0 0 ${radians(-90)}"/>
+      <origin xyz="0 0 0.008" rpy="0 0 ${radians(-90)}"/>
     </xacro:robotiq_hande>
     <!--If statements for the various types of gripper fingers-->
