Commit message: exposed finger selection xacro arguments, updated view_robot.launch.py to suppport testing finger selection

File: chonkur_description/urdf/chonkur.urdf.xacro (robot description, xacro)
@@ -5,4 +5,5 @@
   <xacro:arg name="headless_mode" default="false" />
   <xacro:arg name="ros2_control_name" default="chonkur"/>
+  <xacro:arg name="finger_xacro" default="fngr_v2_m"/>
   <xacro:include filename="$(find chonkur_description)/urdf/chonkur_macro.xacro"/>
   <link name="world" />
@@ -12,4 +13,5 @@
     headless_mode="$(arg headless_mode)"
     ros2_control_name="$(arg ros2_control_name)"
+    finger_xacro="$(arg finger_xacro)"
     parent="world"
     sim_gazebo="false"

File: chonkur_description/urdf/chonkur_macro.xacro (robot description, xacro)
@@ -1,6 +1,7 @@
 <?xml version="1.0"?>
 <robot xmlns:xacro="http://wiki.ros.org/xacro">
-  <!-- import main macro -->
+  <!-- import macros -->
   <xacro:include filename="$(find ur_description)/urdf/ur_macro.xacro"/>
+  <xacro:include filename="$(find dextivr_hande_description)/urdf/dextivr_hande.xacro"/>
   <!-- trying to reuse ur control launch files. So cannot pass in any additional args to the xacro.-->
   <xacro:macro name="chonkur" params="
@@ -13,5 +14,6 @@
     sim_ignition:=false
     chonkur_ip:=192.168.1.102
-    com_port_hande:=/dev/ttyUSB1">
+    com_port_hande:=/dev/ttyUSB1
+    finger_xacro:=fngr_v2_m">
     <!-- convert to property to use substitution in function -->
     <xacro:property name="initial_positions_file" default="$(find chonkur_description)/config/initial_positions.yaml"/>
@@ -81,21 +83,7 @@
       <origin xyz="0 0 0" rpy="0 0 ${radians(90)}"/>
     </xacro:endeff_stack>
-    <xacro:property name="finger_type_prop" value="fngr_v2_m" />
-    <xacro:include filename="$(find robotiq_hande_description)/urdf/robotiq_hande.xacro"/>
-    <xacro:robotiq_hande name="chonkur_hande" tf_prefix="${tf_prefix}" parent="${tf_prefix}ur_realsense_mount" use_fake_hardware="${use_fake_hardware}" com_port="${com_port_hande}">
+    <xacro:dextivr_hande name="dextivr_hande" tf_prefix="${tf_prefix}" parent="${tf_prefix}ur_realsense_mount" use_fake_hardware="${use_fake_hardware}" com_port="${com_port_hande}" finger_xacro="${finger_xacro}">
       <origin xyz="0 0 0.008" rpy="0 0 ${radians(-90)}"/>
-    </xacro:robotiq_hande>
-    <!--If statements for the various types of gripper fingers-->
-    <xacro:if value="${finger_type_prop == 'fngr_nail_v2'}">
-      <xacro:include filename="$(find dextivr_hande_description)/urdf/hande_fingers_fngr_nail_v2.xacro"/>
-      <xacro:include filename="$(find dextivr_hande_description)/urdf/fngr_nail_v2_grasp_push_frames.xacro"/>
-    </xacro:if>
-    <xacro:if value="${finger_type_prop == 'fngr_v2_m'}">
-      <xacro:include filename="$(find dextivr_hande_description)/urdf/hande_fingers_v2_m.xacro"/>
-      <xacro:include filename="$(find dextivr_hande_description)/urdf/fngr_v2_m_grasp_push_frames.xacro"/>
-    </xacro:if>
-    <!--Run the xacros from the files included above-->
-    <xacro:hande_fingers name="chonkur_hande_fingers" tf_prefix="${tf_prefix}"/>
-    <xacro:grasp_push_frames name="chonkur_grasp_push_frames" tf_prefix="${tf_prefix}"/>
+    </xacro:dextivr_hande>
     <link name="manual_grasp_link" />
     <joint name="${tf_prefix}temp_studio_joint" type="fixed">
