Commit message: switched from file to package

File: chonkur_description/urdf/endeff_stack_macro.xacro (robot description, xacro)
@@ -14,5 +14,5 @@
         <visual>
             <geometry>
-                <mesh filename= "file://$(find chonkur_description)/meshes/visual/mtc_robot_side.dae"/>
+                <mesh filename= "package://chonkur_description/meshes/visual/mtc_robot_side.dae"/>
             </geometry>
         </visual>
@@ -26,5 +26,5 @@
         <visual>
             <geometry>
-                <mesh filename= "file://$(find chonkur_description)/meshes/visual/mtc_effector_side.dae"/>
+                <mesh filename= "package://chonkur_description/meshes/visual/mtc_effector_side.dae"/>
             </geometry>
         </visual>
@@ -38,5 +38,5 @@
         <visual>
             <geometry>
-                <mesh filename= "file://$(find chonkur_description)/meshes/visual/ur_realsense_mount.dae"/>
+                <mesh filename= "package://chonkur_description/meshes/visual/ur_realsense_mount.dae"/>
             </geometry>
         </visual>
@@ -50,5 +50,5 @@
         <visual>
             <geometry>
-                <mesh filename= "file://$(find chonkur_description)/meshes/visual/robotiq_hand-e_adapter_old.dae"/>
+                <mesh filename= "package://chonkur_description/meshes/visual/robotiq_hand-e_adapter_old.dae"/>
             </geometry>
         </visual>

Commit message: updated mtc_effector_side to ur_realsense_mount joint origin

File: chonkur_description/urdf/endeff_stack_macro.xacro (robot description, xacro)
@@ -33,5 +33,5 @@
         <parent link="${tf_prefix}mtc_effector_side"/>
         <child link="${tf_prefix}ur_realsense_mount"/>
-        <origin xyz="0 0 0.018684" rpy="0 0 0"/>
+        <origin xyz="0 0 0.023684" rpy="0 0 0"/>
     </joint>
     <link name="${tf_prefix}ur_realsense_mount">

Commit message: updated realsense to hand-e adapter joint origin

File: chonkur_description/urdf/endeff_stack_macro.xacro (robot description, xacro)
@@ -45,5 +45,5 @@
         <parent link="${tf_prefix}ur_realsense_mount"/>
         <child link="${tf_prefix}robotiq_hand-e_adapter_old"/>
-        <origin xyz="0 0 0.006" rpy="0 0 0"/>
+        <origin xyz="0 0 0.003" rpy="0 0 0"/>
     </joint>
     <link name="${tf_prefix}robotiq_hand-e_adapter_old">

Commit message: Camera calibration offsets applied

File: chonkur_description/urdf/endeff_stack_macro.xacro (robot description, xacro)
@@ -42,4 +42,9 @@
         </visual>
     </link>
+    <!-- Realsense camera -->
+    <xacro:include filename="$(find realsense2_description)/urdf/_d435.urdf.xacro"/>
+    <xacro:sensor_d435 parent="${tf_prefix}ur_realsense_mount" use_nominal_extrinsics="true" use_mesh="true">
+        <origin xyz="-0.075 -0.006 0.023" rpy="0.022 -1.386 -0.012"/>
+    </xacro:sensor_d435>
     <joint name="${tf_prefix}realsense_mount_to_hand-e_adapter" type="fixed">
         <parent link="${tf_prefix}ur_realsense_mount"/>

Commit message: corrected camera calibration to use bottom_screw origin

File: chonkur_description/urdf/endeff_stack_macro.xacro (robot description, xacro)
@@ -45,5 +45,5 @@
     <xacro:include filename="$(find realsense2_description)/urdf/_d435.urdf.xacro"/>
     <xacro:sensor_d435 parent="${tf_prefix}ur_realsense_mount" use_nominal_extrinsics="true" use_mesh="true">
-        <origin xyz="-0.075 -0.006 0.023" rpy="0.022 -1.386 -0.012"/>
+        <origin xyz="-0.065 -0.006 0.010" rpy="0.048 -1.392 -0.047"/>
     </xacro:sensor_d435>
     <joint name="${tf_prefix}realsense_mount_to_hand-e_adapter" type="fixed">

Commit message: Adding the new camera mount.

File: chonkur_description/urdf/endeff_stack_macro.xacro (robot description, xacro)
@@ -38,5 +38,5 @@
         <visual>
             <geometry>
-                <mesh filename= "package://chonkur_description/meshes/visual/ur_realsense_mount.dae"/>
+                <mesh filename= "package://chonkur_description/meshes/visual/ur_realsense_short_mount_tube.stl"/>
             </geometry>
         </visual>

Commit message: Adding collisions.

File: chonkur_description/urdf/endeff_stack_macro.xacro (robot description, xacro)
@@ -17,4 +17,9 @@
             </geometry>
         </visual>
+        <collision>
+            <geometry>
+                <mesh filename= "package://chonkur_description/meshes/visual/mtc_robot_side.dae"/>
+            </geometry>
+        </collision>
     </link>
     <joint name="${tf_prefix}mtc_robot_to_effector_side_joint" type="fixed">
@@ -29,4 +34,9 @@
             </geometry>
         </visual>
+        <collision>
+            <geometry>
+                <mesh filename= "package://chonkur_description/meshes/visual/mtc_effector_side.dae"/>
+            </geometry>
+        </collision>
     </link>
     <joint name="${tf_prefix}mtc_effector_side_to_realsense_mount" type="fixed">
@@ -41,4 +51,9 @@
             </geometry>
         </visual>
+        <collision>
+            <geometry>
+                <mesh filename= "package://chonkur_description/meshes/visual/ur_realsense_short_mount_tube.stl"/>
+            </geometry>
+        </collision>
     </link>
     <!-- Realsense camera -->

Commit message: disabling collision for MTC due to failure of servo

File: chonkur_description/urdf/endeff_stack_macro.xacro (robot description, xacro)
@@ -17,9 +17,9 @@
             </geometry>
         </visual>
-        <collision>
+        <!-- <collision>
             <geometry>
                 <mesh filename= "package://chonkur_description/meshes/visual/mtc_robot_side.dae"/>
             </geometry>
-        </collision>
+        </collision> -->
     </link>
     <joint name="${tf_prefix}mtc_robot_to_effector_side_joint" type="fixed">

Commit message: added collisions for quick disconnect

File: chonkur_description/urdf/endeff_stack_macro.xacro (robot description, xacro)
@@ -22,4 +22,10 @@
             </geometry>
         </collision> -->
+        <collision>
+            <geometry>
+                <cylinder length="0.0184" radius="0.0525" />
+            </geometry>
+            <origin xyz="0 0 0.0092" rpy="0 0 0" />
+        </collision>
     </link>
     <joint name="${tf_prefix}mtc_robot_to_effector_side_joint" type="fixed">
@@ -36,6 +42,7 @@
         <collision>
             <geometry>
-                <mesh filename= "package://chonkur_description/meshes/visual/mtc_effector_side.dae"/>
+                <cylinder length="0.0237" radius="0.0525" />
             </geometry>
+            <origin xyz="0 0 0.01185" rpy="0 0 0" />
         </collision>
     </link>

Commit message: camera calibration for freshly printed rigid mount

File: chonkur_description/urdf/endeff_stack_macro.xacro (robot description, xacro)
@@ -60,5 +60,5 @@
     <xacro:include filename="$(find realsense2_description)/urdf/_d435.urdf.xacro"/>
     <xacro:sensor_d435 parent="${tf_prefix}ur_realsense_mount" use_nominal_extrinsics="true" use_mesh="true" name="wrist_mounted_camera">
-        <origin xyz="-0.065 -0.006 0.010" rpy="0.048 -1.392 -0.047"/>
+        <origin xyz="-0.064 -0.003 0.016" rpy="0.136 -1.429 -0.128"/>
     </xacro:sensor_d435>
     </xacro:macro>

Commit message: updated collisions for the quick disconnect

File: chonkur_description/urdf/endeff_stack_macro.xacro (robot description, xacro)
@@ -17,9 +17,4 @@
             </geometry>
         </visual>
-        <!-- <collision>
-            <geometry>
-                <mesh filename= "package://chonkur_description/meshes/visual/mtc_robot_side.dae"/>
-            </geometry>
-        </collision> -->
         <collision>
             <geometry>

Commit message: Avoid Error: material 'aluminum' is not unique

File: chonkur_description/urdf/endeff_stack_macro.xacro (robot description, xacro)
@@ -60,4 +60,5 @@
     </link>
     <!-- Realsense camera -->
+    <xacro:property name="realsense_materials_defined" default="true" />
     <xacro:include filename="$(find realsense2_description)/urdf/_d435.urdf.xacro"/>
     <xacro:sensor_d435 parent="${tf_prefix}ur_realsense_mount" use_nominal_extrinsics="true" use_mesh="true" name="wrist_mounted_camera">

Commit message: set realsense_materials_defined instead of defining default

File: chonkur_description/urdf/endeff_stack_macro.xacro (robot description, xacro)
@@ -60,5 +60,5 @@
     </link>
     <!-- Realsense camera -->
-    <xacro:property name="realsense_materials_defined" default="true" />
+    <xacro:property name="realsense_materials_defined" value="true" />
     <xacro:include filename="$(find realsense2_description)/urdf/_d435.urdf.xacro"/>
     <xacro:sensor_d435 parent="${tf_prefix}ur_realsense_mount" use_nominal_extrinsics="true" use_mesh="true" name="wrist_mounted_camera">
