Commit message: Fix colors and views in materials

File: chonkur/chonkur_description/urdf/endeff_stack_macro.xacro (robot description, xacro)
@@ -52,4 +52,7 @@
                 <mesh filename= "package://chonkur_description/meshes/visual/ur_realsense_short_mount_tube.stl"/>
             </geometry>
+            <material name="${tf_prefix}ur_realsense_mount">
+                <color rgba="0.1 0.1 0.1 1.0"/>
+            </material>
         </visual>
         <collision>

File: clr_description/urdf/clr_macro.xacro (robot description, xacro)
@@ -118,5 +118,5 @@
           <box size="0.05 0.05 0.381"/>
         </geometry>
-        <!-- <material name="safety_light_blue" />         -->
+        <material name="safety_light_blue" />
       </visual>
       <collision>
@@ -136,5 +136,5 @@
           <box size="0.05 0.05 0.381"/>
         </geometry>
-        <!-- <material name="safety_light_blue" />         -->
+        <material name="safety_light_blue" />
       </visual>
       <collision>

File: clr_description/urdf/lift_camera.macro.xacro (robot description, xacro)
@@ -19,5 +19,7 @@
                 <mesh filename= "package://clr_description/meshes/visual/lift_camera_mount.stl"/>
             </geometry>
-            <color rgba="0.1 0.1 0.1 1"/>
+            <material name="${tf_prefix}lift_camera_mount">
+                <color rgba="0.8 0.8 0.8 1"/>
+            </material>
         </visual>
         <collision>

File: clr_description/urdf/plates.macro.xacro (robot description, xacro)
@@ -18,4 +18,7 @@
                     <box size="0.310 0.310 0.01905"/>
                 </geometry>
+                <material name="${tf_prefix}lower_lift_plate">
+                    <color rgba="0.8 0.8 0.8 1"/>
+                </material>
             </visual>
             <collision>
@@ -42,4 +45,7 @@
                     <box size="0.225 0.225 0.01905"/>
                 </geometry>
+                <material name="${tf_prefix}upper_lift_plate">
+                    <color rgba="0.8 0.8 0.8 1"/>
+                </material>
             </visual>
             <collision>
