Commit message: remove manual_grasp_link and temp_studio_joint to fix prefixing issue

File: chonkur/chonkur_description/urdf/chonkur_macro.xacro (robot description, xacro)
@@ -97,10 +97,4 @@
       <origin xyz="0 0 0.008" rpy="0 0 ${radians(-90)}"/>
     </xacro:dextivr_hande>
-    <link name="manual_grasp_link" />
-    <joint name="${tf_prefix}temp_studio_joint" type="fixed">
-      <parent link="${tf_prefix}grasp_frame"/>
-      <child link="${tf_prefix}manual_grasp_link"/>
-      <origin xyz="0 0 0" rpy="0 0 ${radians(180)}"/>
-    </joint>
   </xacro:macro>
 </robot>

Commit message: hardware changes, wrist and lift cameras swapped, end effector stack flipped due to rs485 adapter

File: chonkur/chonkur_description/urdf/chonkur_macro.xacro (robot description, xacro)
@@ -85,5 +85,5 @@
       tf_prefix="${tf_prefix}"
       parent="${tf_prefix}tool0">
-      <origin xyz="0 0 0" rpy="0 0 ${radians(90)}"/>
+      <origin xyz="0 0 0" rpy="0 0 ${radians(-90)}"/>
     </xacro:endeff_stack>
     <xacro:dextivr_hande

Commit message: Rotate the gripper

File: chonkur/chonkur_description/urdf/chonkur_macro.xacro (robot description, xacro)
@@ -97,5 +97,5 @@
       add_grasp_push_frames="${add_grasp_push_frames}"
       generate_ros2_control_tag="${generate_ros2_control_tag}">
-      <origin xyz="0 0 0.008" rpy="0 0 ${radians(-90)}"/>
+      <origin xyz="0 0 0.008" rpy="0 0 ${radians(90)}"/>
     </xacro:dextivr_hande>
   </xacro:macro>

Commit message: matching xacro rotation to hardware after change to thru-arm rs485 wiring

File: chonkur/chonkur_description/urdf/chonkur_macro.xacro (robot description, xacro)
@@ -106,5 +106,5 @@
       add_grasp_push_frames="${add_grasp_push_frames}"
       generate_ros2_control_tag="${generate_ros2_control_tag}">
-      <origin xyz="0 0 0.008" rpy="0 0 ${radians(-90)}"/>
+      <origin xyz="0 0 0.008" rpy="0 0 ${radians(90)}"/>
     </xacro:dextivr_hande>
   </xacro:macro>

File: chonkur/chonkur_description/urdf/endeff_stack_macro.xacro (robot description, xacro)
@@ -45,5 +45,5 @@
         <parent link="${tf_prefix}mtc_effector_side"/>
         <child link="${tf_prefix}ur_realsense_mount"/>
-        <origin xyz="0 0 0.023684" rpy="0 0 0"/>
+        <origin xyz="0 0 0.023684" rpy="0 0 ${radians(180)}"/>
     </joint>
     <link name="${tf_prefix}ur_realsense_mount">
