Commit message: Namespace the multi hatch viewing launchfile

File: urdf/clr_trainer_multi_hatch.urdf.xacro (robot description, xacro)
@@ -22,23 +22,4 @@
   <xacro:property name="second_trainer" value="false"/>
   <link name="world" />
-  <xacro:clr
-    tf_prefix="$(arg tf_prefix)"
-    use_fake_hardware="$(arg use_fake_hardware)"
-    headless_mode="$(arg headless_mode)"
-    ewellix_com_port="$(arg ewellix_com_port)"
-    com_port_hande="$(arg com_port_hande)"
-    finger_xacro="$(arg finger_xacro)"
-    ros2_control_name="clr"
-    parent="world"
-    sim_gazebo="false"
-    sim_ignition="false"
-    chonkur_ip="192.168.1.102"
-    rail_ip="192.168.7.2"
-    rail_port="9999"
-    rail_position_limit="2.0"
-    rail_velocity_limit="0.15"
-    ewellix_height_limit="0.7"
-    safety_com_port="/dev/safety_com_port"
-  />
   <!-- Load the 4040 hatch-->
   <xacro:if value="${hatch_4040}">
@@ -211,5 +192,5 @@
   </link>
   <joint name="ground_joint" type="fixed">
-    <parent link="$(arg tf_prefix)clr_base"/>
+    <parent link="$(arg tf_prefix)world"/>
     <child link="ground_plane"/>
     <origin xyz="0 0 -0.005" rpy="0 0 0"/>
@@ -238,5 +219,5 @@
   </link>
   <joint name="room_ceiling_joint" type="fixed">
-    <parent link="$(arg tf_prefix)clr_base"/>
+    <parent link="$(arg tf_prefix)world"/>
     <child link="room_ceiling"/>
     <origin xyz="0 0 2.75" rpy="0 0 0"/>

Commit message: bring clr into environment. still need to check if args get passed

File: urdf/clr_trainer_multi_hatch.urdf.xacro (robot description, xacro)
@@ -1,4 +1,4 @@
 <?xml version="1.0"?>
-<robot xmlns:xacro="http://wiki.ros.org/xacro" name="clr">
+<robot xmlns:xacro="http://wiki.ros.org/xacro" name="imetro_env">
   <xacro:arg name="name" default=""/>
   <xacro:arg name="tf_prefix" default="" />
@@ -9,5 +9,5 @@
   <xacro:arg name="ewellix_com_port" default="/dev/ewellix" />
   <xacro:arg name="finger_xacro" default="fngr_v2_m" />
-  <xacro:include filename="$(find clr_description)/urdf/clr_macro.xacro"/>
+  <xacro:include filename="$(find clr_description)/urdf/clr.urdf.xacro"/>
   <xacro:include filename="$(find clr_imetro_environments)/urdf/colors.xacro"/>
   <xacro:include filename="$(find clr_imetro_environments)/urdf/long_bench.xacro"/>
@@ -21,5 +21,4 @@
   <xacro:property name="hatch_4060" default="true"/>
   <xacro:property name="second_trainer" value="false"/>
-  <link name="world" />
   <!-- Load the 4040 hatch-->
   <xacro:if value="${hatch_4040}">

Commit message: partial fix to prefix issue -- some components still not prefixed

File: urdf/clr_trainer_multi_hatch.urdf.xacro (robot description, xacro)
@@ -103,26 +103,26 @@
   </xacro:trainer_frame>
   <xacro:include filename="$(find trainer)/urdf/bench_seat.xacro"/>
-  <xacro:bench_seat name="$(arg name)" prefix="$(arg prefix)" parent="trainer_frame">
+  <xacro:bench_seat name="$(arg name)" prefix="$(arg prefix)" parent="$(arg tf_prefix)trainer_frame">
     <origin xyz="1.261 0 0.4769" rpy="0 0 0"/>
   </xacro:bench_seat>
   <xacro:if value="${ceiling_prop}">
     <xacro:include filename="$(find trainer)/urdf/ceiling.xacro"/>
-    <xacro:ceiling name="$(arg name)" prefix="$(arg prefix)" parent="trainer_frame">
+    <xacro:ceiling name="$(arg name)" prefix="$(arg prefix)" parent="$(arg tf_prefix)trainer_frame">
       <origin xyz="0.0 0.0 1.6002" rpy="0 0 0"/>
     </xacro:ceiling>
   </xacro:if>
   <xacro:include filename="$(find trainer)/urdf/trainer_front_left_face.xacro"/>
-  <xacro:trainer_front_left_face name="$(arg name)" prefix="$(arg prefix)" parent="trainer_frame" shelf="${shelf}">
+  <xacro:trainer_front_left_face name="$(arg name)" prefix="$(arg prefix)" parent="$(arg tf_prefix)trainer_frame" shelf="${shelf}">
     <origin xyz="1.25 0.08 0.457" rpy="0 0 0"/>
   </xacro:trainer_front_left_face>
   <xacro:include filename="$(find trainer)/urdf/trainer_front_right_face.xacro"/>
-  <xacro:trainer_front_right_face name="$(arg name)" prefix="$(arg prefix)" parent="trainer_frame">
+  <xacro:trainer_front_right_face name="$(arg name)" prefix="$(arg prefix)" parent="$(arg tf_prefix)trainer_frame">
     <origin xyz="1.25 0.465 0.457" rpy="0 0 0"/>
   </xacro:trainer_front_right_face>
   <xacro:include filename="$(find trainer)/urdf/trainer_side.xacro"/>
-  <xacro:side_face name="$(arg name)" prefix="$(arg prefix)" parent="trainer_frame">
+  <xacro:side_face name="$(arg name)" prefix="$(arg prefix)" parent="$(arg tf_prefix)trainer_frame">
     <origin xyz="0.812 0.887 0.04" rpy="0 0 0"/>
   </xacro:side_face>
-  <xacro:if value="${second_trainer}">
+  <!-- <xacro:if value="${second_trainer}">
     <xacro:trainer_frame name="$(arg name)" prefix="second_trainer/" parent="world">
       <origin xyz="${-0.9 - 1.2192 + 0.02 + 1.1} ${1.8596 + 0.58} 0.0" rpy="0 0 4.7112"/>
@@ -140,5 +140,5 @@
       <origin xyz="0.812 0.887 0.04" rpy="0 0 0"/>
     </xacro:side_face>
-  </xacro:if>
+  </xacro:if> -->
   <!-- long bench
   <xacro:include filename="$(find clr_imetro_environments)/urdf/long_bench.xacro"/>
@@ -147,10 +147,10 @@
   </xacro:long_bench_seat> -->
   <!--This is for when there is a bench at the level of the bottom of the hatch opening.-->
-  <joint name="hatch_level_bench_joint" type="fixed">
-    <parent link="bench_back"/>
-    <child link="hatch_level_bench"/>
+  <joint name="$(arg tf_prefix)hatch_level_bench_joint" type="fixed">
+    <parent link="$(arg tf_prefix)bench_back"/>
+    <child link="$(arg tf_prefix)hatch_level_bench"/>
     <origin xyz="0.706 0.895 0.0" rpy="0 0 0"/>
   </joint>
-  <link name="hatch_level_bench">
+  <link name="$(arg tf_prefix)hatch_level_bench">
     <visual>
       <origin xyz="${-1.2192/2} ${1.193/2} ${0.0527/2}" rpy="0 0 0"/>
@@ -169,5 +169,5 @@
   </link>
   <!-- Plane -->
-  <link name="ground_plane">
+  <link name="$(arg tf_prefix)ground_plane">
     <visual>
         <geometry>
@@ -190,11 +190,11 @@
     </inertial>
   </link>
-  <joint name="ground_joint" type="fixed">
-    <parent link="$(arg tf_prefix)world"/>
-    <child link="ground_plane"/>
+  <joint name="$(arg tf_prefix)ground_joint" type="fixed">
+    <parent link="world"/>
+    <child link="$(arg tf_prefix)ground_plane"/>
     <origin xyz="0 0 -0.005" rpy="0 0 0"/>
   </joint>
   <!-- Plane -->
-  <link name="room_ceiling">
+  <link name="$(arg tf_prefix)room_ceiling">
       <visual>
           <geometry>
@@ -217,7 +217,7 @@
       </inertial>
   </link>
-  <joint name="room_ceiling_joint" type="fixed">
-    <parent link="$(arg tf_prefix)world"/>
-    <child link="room_ceiling"/>
+  <joint name="$(arg tf_prefix)room_ceiling_joint" type="fixed">
+    <parent link="world"/>
+    <child link="$(arg tf_prefix)room_ceiling"/>
     <origin xyz="0 0 2.75" rpy="0 0 0"/>
   </joint>

Commit message: make clr optional

File: urdf/clr_trainer_multi_hatch.urdf.xacro (robot description, xacro)
@@ -9,5 +9,5 @@
   <xacro:arg name="ewellix_com_port" default="/dev/ewellix" />
   <xacro:arg name="finger_xacro" default="fngr_v2_m" />
-  <xacro:include filename="$(find clr_description)/urdf/clr.urdf.xacro"/>
+  <xacro:arg name="include_clr" default="true" />
   <xacro:include filename="$(find clr_imetro_environments)/urdf/colors.xacro"/>
   <xacro:include filename="$(find clr_imetro_environments)/urdf/long_bench.xacro"/>
@@ -15,4 +15,12 @@
   <xacro:include filename="$(find hatch_accessories)/urdf/hatch_frame.xacro"/>
   <xacro:include filename="$(find trainer)/urdf/trainer_frame.xacro"/>
+  <!-- Optionally include CLR -->
+  <xacro:property name="clr" default="$(arg include_clr)"/>
+  <xacro:if value="${clr}">
+    <xacro:include filename="$(find clr_description)/urdf/clr.urdf.xacro"/>
+  </xacro:if>
+  <xacro:if value="${not clr}">
+    <link name="world" />
+  </xacro:if>
   <xacro:property name="shelf" default="false"/>
   <xacro:property name="ceiling_prop" value="false"/>

Commit message: add mockup configuration properties as args

File: urdf/clr_trainer_multi_hatch.urdf.xacro (robot description, xacro)
@@ -9,5 +9,21 @@
   <xacro:arg name="ewellix_com_port" default="/dev/ewellix" />
   <xacro:arg name="finger_xacro" default="fngr_v2_m" />
-  <xacro:arg name="include_clr" default="true" />
+  <!-- Optional includes -->
+  <xacro:arg name="clr" default="true" />
+  <xacro:arg name="shelf" default="false"/>
+  <xacro:arg name="ceiling_prop" default="false"/>
+  <xacro:arg name="hatch_4040" default="false"/>
+  <xacro:arg name="express_rack" default="true"/>
+  <xacro:arg name="hatch_4060" default="true"/>
+  <xacro:arg name="second_trainer" default="false"/>
+  <!-- Convert some args to properties for flexibility -->
+  <xacro:property name="clr" value="$(arg clr)"/>
+  <xacro:property name="shelf" value="$(arg shelf)"/>
+  <xacro:property name="ceiling_prop" value="$(arg ceiling_prop)"/>
+  <xacro:property name="hatch_4040" value="$(arg hatch_4040)"/>
+  <xacro:property name="express_rack" value="$(arg express_rack)"/>
+  <xacro:property name="hatch_4060" value="$(arg hatch_4060)"/>
+  <xacro:property name="second_trainer" value="$(arg second_trainer)"/>
+  <!-- Include xacros -->
   <xacro:include filename="$(find clr_imetro_environments)/urdf/colors.xacro"/>
   <xacro:include filename="$(find clr_imetro_environments)/urdf/long_bench.xacro"/>
@@ -15,6 +31,5 @@
   <xacro:include filename="$(find hatch_accessories)/urdf/hatch_frame.xacro"/>
   <xacro:include filename="$(find trainer)/urdf/trainer_frame.xacro"/>
-  <!-- Optionally include CLR -->
-  <xacro:property name="clr" default="$(arg include_clr)"/>
+  <!-- Load CLR as urdf to use default CLR macro config-->
   <xacro:if value="${clr}">
     <xacro:include filename="$(find clr_description)/urdf/clr.urdf.xacro"/>
@@ -23,10 +38,4 @@
     <link name="world" />
   </xacro:if>
-  <xacro:property name="shelf" default="false"/>
-  <xacro:property name="ceiling_prop" value="false"/>
-  <xacro:property name="hatch_4040" default="false"/>
-  <xacro:property name="express_rack" default="true"/>
-  <xacro:property name="hatch_4060" default="true"/>
-  <xacro:property name="second_trainer" value="false"/>
   <!-- Load the 4040 hatch-->
   <xacro:if value="${hatch_4040}">

Commit message: use clr macro instead of urdf now that defaults have been updated

File: urdf/clr_trainer_multi_hatch.urdf.xacro (robot description, xacro)
@@ -5,7 +5,6 @@
   <xacro:arg name="use_fake_hardware" default="false" />
   <xacro:arg name="headless_mode" default="false" />
-  <xacro:arg name="com_port_hande" default="/dev/robotiq" />
-  <xacro:arg name="ewellix_com_port" default="/dev/ewellix" />
   <xacro:arg name="finger_xacro" default="fngr_v6" />
+  <xacro:arg name="generate_ros2_control_tag" default="true" />
   <!-- Optional includes -->
   <xacro:arg name="clr" default="true" />
@@ -25,4 +24,5 @@
   <xacro:property name="second_trainer" value="$(arg second_trainer)"/>
   <!-- Include xacros -->
+  <xacro:include filename="$(find clr_description)/urdf/clr_macro.xacro"/>
   <xacro:include filename="$(find clr_imetro_environments)/urdf/colors.xacro"/>
   <xacro:include filename="$(find clr_imetro_environments)/urdf/long_bench.xacro"/>
@@ -30,10 +30,14 @@
   <xacro:include filename="$(find hatch_accessories)/urdf/hatch_frame.xacro"/>
   <xacro:include filename="$(find trainer)/urdf/trainer_frame.xacro"/>
-  <!-- Load CLR as urdf to use default CLR macro config-->
+  <link name="world" />
+  <!-- Load CLR -->
   <xacro:if value="${clr}">
-    <xacro:include filename="$(find clr_description)/urdf/clr.urdf.xacro"/>
-  </xacro:if>
-  <xacro:if value="${not clr}">
-    <link name="world" />
+    <xacro:clr
+      tf_prefix="$(arg tf_prefix)"
+      use_fake_hardware="$(arg use_fake_hardware)"
+      headless_mode="$(arg headless_mode)"
+      finger_xacro="$(arg finger_xacro)"
+      generate_ros2_control_tag="$(arg generate_ros2_control_tag)"
+    />
   </xacro:if>
   <!-- Load the 4040 hatch-->
