Commit message: Make 4060 hatch latch go away on HW

File: clr_imetro_environments/urdf/clr_trainer_multi_hatch.urdf.xacro (robot description, xacro)
@@ -12,4 +12,5 @@
   <xacro:arg name="express_rack" default="true"/>
   <xacro:arg name="hatch_4060" default="true"/>
+  <xacro:arg name="hatch_4060_latch" default="false"/>
   <xacro:arg name="second_trainer" default="false"/>
   <xacro:arg name="add_localization_joints" default="false"/>
@@ -26,4 +27,5 @@
     ceiling_prop="$(arg ceiling_prop)"
     hatch_4040="$(arg hatch_4040)"
+    hatch_4060_latch="$(arg hatch_4060_latch)"
     express_rack="$(arg express_rack)"
     hatch_4060="$(arg hatch_4060)"

File: clr_imetro_environments/urdf/clr_trainer_multi_hatch_macro.xacro (robot description, xacro)
@@ -15,4 +15,5 @@
     express_rack:=true
     hatch_4060:=true
+    hatch_4060_latch:=false
     second_trainer:=false
     add_localization_joints:=false
@@ -96,9 +97,8 @@
       <xacro:property name="internal_handle_1" default="false"/>
       <xacro:property name="internal_handle_2" default="true"/>
-      <xacro:property name="latch" default="true"/>
       <xacro:include filename="$(find hatch_4060)/urdf/hatch_4060.xacro"/>
       <xacro:hatch_4060 prefix="lorge/" parent="lorge/hatch_frame"
         external_handle_1="${external_handle_1}" external_handle_2="${external_handle_2}" external_handle_3="${external_handle_3}"
-        internal_handle_1="${internal_handle_1}" internal_handle_2="${internal_handle_2}" latch="${latch}">
+        internal_handle_1="${internal_handle_1}" internal_handle_2="${internal_handle_2}" latch="$(arg hatch_4060_latch)">
         <!-- <origin xyz="${0.678 + 0.012} 0.057 ${0.716 - 0.013}" rpy="0 0 0"/> -->
         <origin xyz="0.678 0.057 0.716" rpy="0 0 0"/>
