Commit message: Adding dynamics to all of the joints for friction and damping

File: clr_imetro_environments/urdf/long_bench.xacro (robot description, xacro)
@@ -100,4 +100,5 @@
       <child link="${prefix}bench_lid"/>
       <origin xyz="0.127 0.0 0.0475" rpy="0 0 0"/>
+      <dynamics friction="3.0" damping="3.0"/>
     </joint>
     <link name="${prefix}bench_lid">
