Commit message: added latch model to mujoco sim, needs more tuning, but works well enough as a latch

File: clr_imetro_environments/urdf/clr_trainer_multi_hatch_macro.xacro (robot description, xacro)
@@ -94,8 +94,9 @@
       <xacro:property name="internal_handle_1" default="false"/>
       <xacro:property name="internal_handle_2" default="true"/>
+      <xacro:property name="latch" default="true"/>
       <xacro:include filename="$(find hatch_4060)/urdf/hatch_4060.xacro"/>
       <xacro:hatch_4060 prefix="lorge/" parent="lorge/hatch_frame"
         external_handle_1="${external_handle_1}" external_handle_2="${external_handle_2}" external_handle_3="${external_handle_3}"
-        internal_handle_1="${internal_handle_1}" internal_handle_2="${internal_handle_2}">
+        internal_handle_1="${internal_handle_1}" internal_handle_2="${internal_handle_2}" latch="${latch}">
         <!-- <origin xyz="${0.678 + 0.012} 0.057 ${0.716 - 0.013}" rpy="0 0 0"/> -->
         <origin xyz="0.678 0.057 0.716" rpy="0 0 0"/>
