Commit message: updating colors

File: clr_imetro_environments/urdf/colors.xacro (robot description, xacro)
@@ -10,4 +10,10 @@
     <color rgba="0 0 1.0 1"/>
   </material>
+  <material name="white">
+    <color rgba="1.0 1.0 1.0 1"/>
+  </material>
+  <material name="aluminum">
+    <color rgba="0.85 0.85 0.85 1"/>
+  </material>
   <material name="gray">
     <color rgba="0.85 0.85 0.85 1.0"/>
