Commit message: added a planning group state

File: clr_moveit_config/srdf/clr_macro.srdf.xacro (robot description, xacro)
@@ -50,4 +50,14 @@
       <joint name="wrist_3_joint" value="-0.11" />
     </group_state>
+    <group_state name="clr_home" group="chonkur_l_raile">
+      <joint name="ewellix_lift_lower_to_higher" value="0.004344256" />
+      <joint name="vention_rail_base_to_carriage" value="0.0"/>
+      <joint name="elbow_joint" value="-2.3058078289031982" />
+      <joint name="shoulder_lift_joint" value="-0.7107666295817872" />
+      <joint name="shoulder_pan_joint" value="3.052349805831909" />
+      <joint name="wrist_1_joint" value="-3.2056271038451136" />
+      <joint name="wrist_2_joint" value="-1.468212906514303" />
+      <joint name="wrist_3_joint" value="0.03171319141983986" />
+    </group_state>
     <!--END EFFECTOR - Purpose - Represent information about an end effector.-->
     <!--VIRTUAL JOINT - Purpose - this element defines a virtual joint between a robot link and an external frame of reference (considered fixed with respect to the robot)-->

Commit message: added gripper to srdf

File: clr_moveit_config/srdf/clr_macro.srdf.xacro (robot description, xacro)
@@ -29,5 +29,22 @@
       <group name="lift" />
     </group>
+    <!-- todo - include push and grasp frames for motion planning-->
+    <!-- end effector - todo abstract out for other grippers -->
+    <group name="hand">
+      <link name="gripper_base_link"/>
+      <link name="finger_1_link"/>
+      <link name="finger_2_link"/>
+      <joint name="finger_1_joint"/>
+      <passive_joint name="finger_2_joint"/>
+    </group>
     <!--GROUP STATES - Purpose - Define a named state for a particular group, in terms of joint values. This is useful to define states like 'folded arms'-->
+    <group_state group="hand" name="open">
+      <joint name="finger_1_joint" value="0.03"/>
+      <joint name="finger_2_joint" value="0.03"/>
+    </group_state>
+    <group_state group="hand" name="close">
+      <joint name="finger_1_joint" value="0"/>
+      <joint name="finger_2_joint" value="0"/>
+    </group_state>
     <group_state name="home" group="ur_manipulator">
       <joint name="elbow_joint" value="0" />
@@ -64,5 +81,5 @@
       <joint name="wrist_3_joint" value="0.03171319141983986" />
     </group_state>
-    <!--END EFFECTOR - Purpose - Represent information about an end effector.-->
+    <end_effector group="hand" name="hand" parent_group="ur_manipulator" parent_link="tool0"/>
     <!--VIRTUAL JOINT - Purpose - this element defines a virtual joint between a robot link and an external frame of reference (considered fixed with respect to the robot)-->
     <!--DISABLE COLLISIONS - By default it is assumed that any link of the robot could potentially come into collision with any other link in the robot. This tag disables collision checking between a specified pair of links. -->

Commit message: add stow position to srdf

File: clr_moveit_config/srdf/clr_macro.srdf.xacro (robot description, xacro)
@@ -70,4 +70,12 @@
         <joint name="wrist_2_joint" value="-1.6" />
         <joint name="wrist_3_joint" value="-0.11" />
+      </group_state>
+      <group_state name="stow" group="ur_manipulator">
+        <joint name="elbow_joint" value="2.44346" />
+        <joint name="shoulder_lift_joint" value="-2.6529" />
+        <joint name="shoulder_pan_joint" value="-2.11185" />
+        <joint name="wrist_1_joint" value="0.0" />
+        <joint name="wrist_2_joint" value="1.0821" />
+        <joint name="wrist_3_joint" value="3.26377" />
       </group_state>
       <group_state name="clr_home" group="clr">

Commit message: Add the grasp frame to the hand group

File: clr_moveit_config/srdf/clr_macro.srdf.xacro (robot description, xacro)
@@ -35,4 +35,5 @@
         <link name="finger_1_link"/>
         <link name="finger_2_link"/>
+        <link name="grasp_frame" />
         <joint name="finger_1_joint"/>
         <passive_joint name="finger_2_joint"/>

Commit message: Reduce finger open states in the SRDF

File: clr_moveit_config/srdf/clr_macro.srdf.xacro (robot description, xacro)
@@ -41,6 +41,6 @@
       <!--GROUP STATES - Purpose - Define a named state for a particular group, in terms of joint values. This is useful to define states like 'folded arms'-->
       <group_state group="hand" name="open">
-        <joint name="finger_1_joint" value="0.03"/>
-        <joint name="finger_2_joint" value="0.03"/>
+        <joint name="finger_1_joint" value="0.025"/>
+        <joint name="finger_2_joint" value="0.025"/>
       </group_state>
       <group_state group="hand" name="close">
