Commit message: handling include_scene_objects arg correctly

File: clr_mujoco_config/urdf/clr_mujoco_processed_inputs.xacro (robot description, xacro)
@@ -1,5 +1,7 @@
 <?xml version="1.0"?>
 <robot xmlns:xacro="http://wiki.ros.org/xacro">
-  <xacro:macro name="clr_mujoco_processed_inputs">
+  <xacro:macro name="clr_mujoco_processed_inputs" params="
+    include_scene_objects:=false
+  ">
     <!-- Process arguments for the URDF -->
     <processed_inputs>
@@ -14,5 +16,7 @@
         <decompose_mesh mesh_name="hatch_4060_frame" threshold="0.05"/>
         <decompose_mesh mesh_name="bench_lid" threshold="0.05"/>
-        <decompose_mesh mesh_name="ctb_handle" threshold="0.01"/>
+        <xacro:if value="${include_scene_objects}">
+          <decompose_mesh mesh_name="ctb_handle" threshold="0.01"/>
+        </xacro:if>
         <!-- The camera with the specified values will be added at the specified site name. -->
         <!-- The position and quaterinion will be filled in by the converter -->

Commit message: Add tf prefixes to mujoco inputs

File: clr_mujoco_config/urdf/clr_mujoco_processed_inputs.xacro (robot description, xacro)
@@ -3,4 +3,5 @@
   <xacro:macro name="clr_mujoco_processed_inputs" params="
     include_scene_objects:=false
+    tf_prefix:=''
   ">
     <!-- Process arguments for the URDF -->
@@ -21,21 +22,21 @@
         <!-- The camera with the specified values will be added at the specified site name. -->
         <!-- The position and quaterinion will be filled in by the converter -->
-        <camera site="wrist_mounted_camera_color_optical_frame" name="wrist_mounted_camera" fovy="58" mode="fixed" resolution="640 480"/>
-        <camera site="lift_camera_color_optical_frame" name="lift_camera" fovy="58" mode="fixed" resolution="640 480"/>
+        <camera site="${tf_prefix}wrist_mounted_camera_color_optical_frame" name="${tf_prefix}wrist_mounted_camera" fovy="58" mode="fixed" resolution="640 480"/>
+        <camera site="${tf_prefix}lift_camera_color_optical_frame" name="${tf_prefix}lift_camera" fovy="58" mode="fixed" resolution="640 480"/>
         <!-- Don't let the merlin open -->
         <modify_element type="joint" name="door_to_frame_joint" range="-0.01 0" />
         <!-- Add gravity compensation for moveable CLR components to improve control -->
-        <modify_element type="body" name="vention_rail_carriage" gravcomp="1.0"/>
-        <modify_element type="body" name="ewellix_lift_higher_link" gravcomp="1.0"/>
-        <modify_element type="body" name="ewellix_lift_middle_link" gravcomp="1.0"/>
-        <modify_element type="body" name="shoulder_link" gravcomp="1.0"/>
-        <modify_element type="body" name="upper_arm_link" gravcomp="1.0"/>
-        <modify_element type="body" name="forearm_link" gravcomp="1.0"/>
-        <modify_element type="body" name="wrist_1_link" gravcomp="1.0"/>
-        <modify_element type="body" name="wrist_2_link" gravcomp="1.0"/>
-        <modify_element type="body" name="wrist_3_link" gravcomp="1.0"/>
+        <modify_element type="body" name="${tf_prefix}vention_rail_carriage" gravcomp="1.0"/>
+        <modify_element type="body" name="${tf_prefix}ewellix_lift_higher_link" gravcomp="1.0"/>
+        <modify_element type="body" name="${tf_prefix}ewellix_lift_middle_link" gravcomp="1.0"/>
+        <modify_element type="body" name="${tf_prefix}shoulder_link" gravcomp="1.0"/>
+        <modify_element type="body" name="${tf_prefix}upper_arm_link" gravcomp="1.0"/>
+        <modify_element type="body" name="${tf_prefix}forearm_link" gravcomp="1.0"/>
+        <modify_element type="body" name="${tf_prefix}wrist_1_link" gravcomp="1.0"/>
+        <modify_element type="body" name="${tf_prefix}wrist_2_link" gravcomp="1.0"/>
+        <modify_element type="body" name="${tf_prefix}wrist_3_link" gravcomp="1.0"/>
         <!-- Add frictionloss and armature to fingers to help with backdriving -->
-        <modify_element type="joint" name="finger_1_joint" armature="0.5" frictionloss="5.0" />
-        <modify_element type="joint" name="finger_2_joint" armature="0.5" frictionloss="5.0" />
+        <modify_element type="joint" name="${tf_prefix}finger_1_joint" armature="0.5" frictionloss="5.0" />
+        <modify_element type="joint" name="${tf_prefix}finger_2_joint" armature="0.5" frictionloss="5.0" />
         <!-- Add joint properties to lorge hatch latch spring joint -->
         <modify_element type="joint" name="lorge/latch_spring" limited="true" springref="0.035" stiffness="10000" damping="2" armature="0.001"/>

File: clr_mujoco_config/urdf/clr_mujoco_raw_inputs.xacro (robot description, xacro)
@@ -1,5 +1,7 @@
 <?xml version="1.0"?>
 <robot xmlns:xacro="http://wiki.ros.org/xacro">
-  <xacro:macro name="clr_mujoco_raw_inputs">
+  <xacro:macro name="clr_mujoco_raw_inputs" params="
+    tf_prefix:=''
+  ">
     <raw_inputs>
         <option integrator="implicitfast"/>
@@ -33,13 +35,13 @@
         </default>
         <actuator>
-            <position joint="vention_rail_base_to_carriage" name="vention_rail_base_to_carriage" kp="25000" dampratio="1.0" ctrlrange="0.0 2.0" />
-            <position joint="ewellix_lift_lower_to_higher" name="ewellix_lift_lower_to_higher" kp="75000" dampratio="1.0" ctrlrange="0.0 0.7" />
-            <position class="size4" name="shoulder_pan_joint" joint="shoulder_pan_joint"/>
-            <position class="size4" name="shoulder_lift_joint" joint="shoulder_lift_joint"/>
-            <position class="size3_limited" name="elbow_joint" joint="elbow_joint"/>
-            <position class="size2" name="wrist_1_joint" joint="wrist_1_joint"/>
-            <position class="size2" name="wrist_2_joint" joint="wrist_2_joint"/>
-            <position class="size2" name="wrist_3_joint" joint="wrist_3_joint"/>
-            <position tendon="split" name="finger_1_joint" kp="10000" dampratio="3.0" ctrlrange="0.0 0.025" forcerange="-100 100"/>
+            <position joint="${tf_prefix}vention_rail_base_to_carriage" name="${tf_prefix}vention_rail_base_to_carriage" kp="25000" dampratio="1.0" ctrlrange="0.0 2.0" />
+            <position joint="${tf_prefix}ewellix_lift_lower_to_higher" name="${tf_prefix}ewellix_lift_lower_to_higher" kp="75000" dampratio="1.0" ctrlrange="0.0 0.7" />
+            <position class="size4" name="${tf_prefix}shoulder_pan_joint" joint="${tf_prefix}shoulder_pan_joint"/>
+            <position class="size4" name="${tf_prefix}shoulder_lift_joint" joint="${tf_prefix}shoulder_lift_joint"/>
+            <position class="size3_limited" name="${tf_prefix}elbow_joint" joint="${tf_prefix}elbow_joint"/>
+            <position class="size2" name="${tf_prefix}wrist_1_joint" joint="${tf_prefix}wrist_1_joint"/>
+            <position class="size2" name="${tf_prefix}wrist_2_joint" joint="${tf_prefix}wrist_2_joint"/>
+            <position class="size2" name="${tf_prefix}wrist_3_joint" joint="${tf_prefix}wrist_3_joint"/>
+            <position tendon="${tf_prefix}split" name="${tf_prefix}finger_1_joint" kp="10000" dampratio="3.0" ctrlrange="0.0 0.025" forcerange="-100 100"/>
         </actuator>
         <!--
@@ -50,33 +52,33 @@
         -->
         <tendon>
-            <fixed name="split">
-            <joint joint="finger_1_joint" coef="0.5"/>
-            <joint joint="finger_2_joint" coef="0.5"/>
+            <fixed name="${tf_prefix}split">
+            <joint joint="${tf_prefix}finger_1_joint" coef="0.5"/>
+            <joint joint="${tf_prefix}finger_2_joint" coef="0.5"/>
             </fixed>
         </tendon>
         <equality>
-            <joint joint1="finger_1_joint" joint2="finger_2_joint" polycoef="0 1 0 0 0" solimp="0.95 0.99 0.001" solref="0.005 1"/>
+            <joint joint1="${tf_prefix}finger_1_joint" joint2="${tf_prefix}finger_2_joint" polycoef="0 1 0 0 0" solimp="0.95 0.99 0.001" solref="0.005 1"/>
         </equality>
         <!-- Same logic as above... -->
         <tendon>
-            <fixed name="lift_middle_mimic_higher">
-            <joint joint="ewellix_lift_lower_to_higher" coef="0.5"/>
-            <joint joint="middle_mimic_higher" coef="0.5"/>
+            <fixed name="${tf_prefix}lift_middle_mimic_higher">
+            <joint joint="${tf_prefix}ewellix_lift_lower_to_higher" coef="0.5"/>
+            <joint joint="${tf_prefix}middle_mimic_higher" coef="0.5"/>
             </fixed>
         </tendon>
         <!-- The mimic joint is scaled by 50% in the URDF -->
         <equality>
-            <joint name="upper_mimic_lower" joint1="ewellix_lift_lower_to_higher" joint2="middle_mimic_higher" polycoef="0 2 0 0 0"/>
+            <joint name="${tf_prefix}upper_mimic_lower" joint1="${tf_prefix}ewellix_lift_lower_to_higher" joint2="${tf_prefix}middle_mimic_higher" polycoef="0 2 0 0 0"/>
         </equality>
         <sensor>
-            <force name="tcp_fts_sensor_force" site="ft_frame"/>
-            <torque name="tcp_fts_sensor_torque" site="ft_frame"/>
+            <force name="${tf_prefix}tcp_fts_sensor_force" site="${tf_prefix}ft_frame"/>
+            <torque name="${tf_prefix}tcp_fts_sensor_torque" site="${tf_prefix}ft_frame"/>
         </sensor>
         <!-- clr contacts -->
         <contact>
-            <exclude body1="world" body2="vention_rail_carriage"/>
-            <exclude body1="world" body2="ewellix_lift_higher_link"/>
-            <exclude body1="world" body2="ewellix_lift_middle_link"/>
-            <exclude body1="vention_rail_carriage" body2="ewellix_lift_middle_link"/>
+            <exclude body1="world" body2="${tf_prefix}vention_rail_carriage"/>
+            <exclude body1="world" body2="${tf_prefix}ewellix_lift_higher_link"/>
+            <exclude body1="world" body2="${tf_prefix}ewellix_lift_middle_link"/>
+            <exclude body1="${tf_prefix}vention_rail_carriage" body2="${tf_prefix}ewellix_lift_middle_link"/>
         </contact>
         <!-- environment contacts -->
