Commit message: Allow inclusion of clr mujoco inputs in other files

File: clr_mujoco_config/urdf/clr_mujoco_processed_inputs.xacro (robot description, xacro)
@@ -1,14 +1,14 @@
 <?xml version="1.0"?>
 <robot xmlns:xacro="http://wiki.ros.org/xacro">
-  <xacro:macro name="clr_mujoco_processed_inputs" params="
+  <xacro:macro name="clr_mujoco_processed_inputs_content" params="
+    model_env:=true
     include_scene_objects:=false
     tf_prefix:=''
   ">
-    <!-- Process arguments for the URDF -->
-    <processed_inputs>
-        <!-- Specifying decompose_mesh will set the `decompose` flag when using obj2mjcf -->
-        <decompose_mesh mesh_name="finger_v6" threshold="0.05"/>
-        <decompose_mesh mesh_name="clr_base" threshold="0.05"/>
-        <!-- env stuff -->
+      <!-- Specifying decompose_mesh will set the `decompose` flag when using obj2mjcf -->
+      <decompose_mesh mesh_name="finger_v6" threshold="0.05"/>
+      <decompose_mesh mesh_name="clr_base" threshold="0.05"/>
+      <!-- env stuff -->
+      <xacro:if value="${model_env}">
         <decompose_mesh mesh_name="crank_wheel" threshold="0.05"/>
         <decompose_mesh mesh_name="imetro_hatch_handle" threshold="0.05"/>
@@ -17,29 +17,53 @@
         <decompose_mesh mesh_name="hatch_4060_frame" threshold="0.05"/>
         <decompose_mesh mesh_name="bench_lid" threshold="0.05"/>
-        <xacro:if value="${include_scene_objects}">
-          <decompose_mesh mesh_name="ctb_handle" threshold="0.01"/>
-        </xacro:if>
-        <!-- The camera with the specified values will be added at the specified site name. -->
-        <!-- The position and quaterinion will be filled in by the converter -->
-        <camera site="${tf_prefix}wrist_mounted_camera_color_optical_frame" name="${tf_prefix}wrist_mounted_camera" fovy="58" mode="fixed" resolution="640 480"/>
-        <camera site="${tf_prefix}lift_camera_color_optical_frame" name="${tf_prefix}lift_camera" fovy="58" mode="fixed" resolution="640 480"/>
-        <!-- Don't let the merlin open -->
-        <modify_element type="joint" name="door_to_frame_joint" range="-0.01 0" />
-        <!-- Add gravity compensation for moveable CLR components to improve control -->
-        <modify_element type="body" name="${tf_prefix}vention_rail_carriage" gravcomp="1.0"/>
-        <modify_element type="body" name="${tf_prefix}ewellix_lift_higher_link" gravcomp="1.0"/>
-        <modify_element type="body" name="${tf_prefix}ewellix_lift_middle_link" gravcomp="1.0"/>
-        <modify_element type="body" name="${tf_prefix}shoulder_link" gravcomp="1.0"/>
-        <modify_element type="body" name="${tf_prefix}upper_arm_link" gravcomp="1.0"/>
-        <modify_element type="body" name="${tf_prefix}forearm_link" gravcomp="1.0"/>
-        <modify_element type="body" name="${tf_prefix}wrist_1_link" gravcomp="1.0"/>
-        <modify_element type="body" name="${tf_prefix}wrist_2_link" gravcomp="1.0"/>
-        <modify_element type="body" name="${tf_prefix}wrist_3_link" gravcomp="1.0"/>
-        <!-- Add frictionloss and armature to fingers to help with backdriving -->
-        <modify_element type="joint" name="${tf_prefix}finger_1_joint" armature="0.5" frictionloss="5.0" />
-        <modify_element type="joint" name="${tf_prefix}finger_2_joint" armature="0.5" frictionloss="5.0" />
-        <!-- Add joint properties to lorge hatch latch spring joint -->
-        <modify_element type="joint" name="lorge/latch_spring" limited="true" springref="0.035" stiffness="10000" damping="2" armature="0.001"/>
-    </processed_inputs>
+      </xacro:if>
+      <xacro:if value="${include_scene_objects}">
+        <decompose_mesh mesh_name="ctb_handle" threshold="0.01"/>
+      </xacro:if>
+      <!-- The camera with the specified values will be added at the specified site name. -->
+      <!-- The position and quaterinion will be filled in by the converter -->
+      <camera site="${tf_prefix}wrist_mounted_camera_color_optical_frame" name="${tf_prefix}wrist_mounted_camera" fovy="58" mode="fixed" resolution="640 480"/>
+      <camera site="${tf_prefix}lift_camera_color_optical_frame" name="${tf_prefix}lift_camera" fovy="58" mode="fixed" resolution="640 480"/>
+      <!-- Don't let the merlin open -->
+      <modify_element type="joint" name="door_to_frame_joint" range="-0.01 0" />
+      <!-- Add gravity compensation for moveable CLR components to improve control -->
+      <modify_element type="body" name="${tf_prefix}vention_rail_carriage" gravcomp="1.0"/>
+      <modify_element type="body" name="${tf_prefix}ewellix_lift_higher_link" gravcomp="1.0"/>
+      <modify_element type="body" name="${tf_prefix}ewellix_lift_middle_link" gravcomp="1.0"/>
+      <modify_element type="body" name="${tf_prefix}shoulder_link" gravcomp="1.0"/>
+      <modify_element type="body" name="${tf_prefix}upper_arm_link" gravcomp="1.0"/>
+      <modify_element type="body" name="${tf_prefix}forearm_link" gravcomp="1.0"/>
+      <modify_element type="body" name="${tf_prefix}wrist_1_link" gravcomp="1.0"/>
+      <modify_element type="body" name="${tf_prefix}wrist_2_link" gravcomp="1.0"/>
+      <modify_element type="body" name="${tf_prefix}wrist_3_link" gravcomp="1.0"/>
+      <!-- Add frictionloss and armature to fingers to help with backdriving -->
+      <modify_element type="joint" name="${tf_prefix}finger_1_joint" armature="0.5" frictionloss="5.0" />
+      <modify_element type="joint" name="${tf_prefix}finger_2_joint" armature="0.5" frictionloss="5.0" />
+      <!-- Add joint properties to lorge hatch latch spring joint -->
+      <modify_element type="joint" name="lorge/latch_spring" limited="true" springref="0.035" stiffness="10000" damping="2" armature="0.001"/>
+  </xacro:macro>
+  <!-- Can use `skip_tags` to include the macro in other files without duplicating inputs -->
+  <xacro:macro name="clr_mujoco_processed_inputs" params="
+    model_env:=true
+    include_scene_objects:=false
+    tf_prefix:=''
+    skip_tags:=false
+  ">
+    <xacro:unless value="${skip_tags}">
+      <processed_inputs>
+        <xacro:clr_mujoco_processed_inputs_content
+          model_env="${model_env}"
+          include_scene_objects="${include_scene_objects}"
+          tf_prefix="${tf_prefix}"
+        />
+      </processed_inputs>
+    </xacro:unless>
+    <xacro:if value="${skip_tags}">
+      <xacro:clr_mujoco_processed_inputs_content
+        model_env="${model_env}"
+        include_scene_objects="${include_scene_objects}"
+        tf_prefix="${tf_prefix}"
+      />
+    </xacro:if>
   </xacro:macro>
 </robot>

File: clr_mujoco_config/urdf/clr_mujoco_raw_inputs.xacro (robot description, xacro)
@@ -1,86 +1,90 @@
 <?xml version="1.0"?>
 <robot xmlns:xacro="http://wiki.ros.org/xacro">
-  <xacro:macro name="clr_mujoco_raw_inputs" params="
+  <xacro:macro name="clr_mujoco_raw_inputs_content" params="
+    model_env:=true
     tf_prefix:=''
+    defaults_prefix:=''
   ">
-    <raw_inputs>
-        <option integrator="implicitfast"/>
-        <default>
+      <option integrator="implicitfast"/>
+      <default>
+        <default class="clr">
             <material specular="0.5" shininess="0.25"/>
             <joint axis="0 1 0" range="-6.28319 6.28319" armature="0.1"/>
             <position ctrlrange="-6.2831 6.2831"/>
             <general biastype="affine" ctrlrange="-6.2831 6.2831" />
-            <default class="size4">
+            <default class="clr_size4">
             <joint damping="10"/>
             <general forcerange="-330 330" gainprm="100000" biasprm="0 -100000 -10000" />
             </default>
-            <default class="size3">
+            <default class="clr_size3">
             <joint damping="5"/>
             <general forcerange="-150 150" gainprm="40000" biasprm="0 -40000 -4000" />
-            <default class="size3_limited">
+            <default class="clr_size3_limited">
                 <joint range="-3.1415 3.1415"/>
                 <general ctrlrange="-3.1415 3.1415" />
             </default>
             </default>
-            <default class="size2">
+            <default class="clr_size2">
             <joint damping="2"/>
             <general forcerange="-56 56" gainprm="10000" biasprm="0 -10000 -1000" />
             </default>
-            <default class="visual">
+            <default class="${defaults_prefix}visual">
             <geom group="2" type="mesh" contype="0" conaffinity="0"/>
             </default>
-            <default class="collision">
+            <default class="${defaults_prefix}collision">
             <geom group="3" type="mesh"/>
-            </default>
+          </default>
         </default>
-        <actuator>
-            <position joint="${tf_prefix}vention_rail_base_to_carriage" name="${tf_prefix}vention_rail_base_to_carriage" kp="25000" dampratio="1.0" ctrlrange="0.0 2.0" />
-            <position joint="${tf_prefix}ewellix_lift_lower_to_higher" name="${tf_prefix}ewellix_lift_lower_to_higher" kp="75000" dampratio="1.0" ctrlrange="0.0 0.7" />
-            <position class="size4" name="${tf_prefix}shoulder_pan_joint" joint="${tf_prefix}shoulder_pan_joint"/>
-            <position class="size4" name="${tf_prefix}shoulder_lift_joint" joint="${tf_prefix}shoulder_lift_joint"/>
-            <position class="size3_limited" name="${tf_prefix}elbow_joint" joint="${tf_prefix}elbow_joint"/>
-            <position class="size2" name="${tf_prefix}wrist_1_joint" joint="${tf_prefix}wrist_1_joint"/>
-            <position class="size2" name="${tf_prefix}wrist_2_joint" joint="${tf_prefix}wrist_2_joint"/>
-            <position class="size2" name="${tf_prefix}wrist_3_joint" joint="${tf_prefix}wrist_3_joint"/>
-            <position tendon="${tf_prefix}split" name="${tf_prefix}finger_1_joint" kp="10000" dampratio="3.0" ctrlrange="0.0 0.025" forcerange="-100 100"/>
-        </actuator>
-        <!--
-            This adds stability to the model by having a tendon that distributes the forces between both
-            joints, such that the equality constraint doesn't have to do that much work in order to equalize
-            both joints. Since both joints share the same sign, we split the force between both equally by
-            setting coef=0.5
-        -->
-        <tendon>
-            <fixed name="${tf_prefix}split">
-            <joint joint="${tf_prefix}finger_1_joint" coef="0.5"/>
-            <joint joint="${tf_prefix}finger_2_joint" coef="0.5"/>
-            </fixed>
-        </tendon>
-        <equality>
-            <joint joint1="${tf_prefix}finger_1_joint" joint2="${tf_prefix}finger_2_joint" polycoef="0 1 0 0 0" solimp="0.95 0.99 0.001" solref="0.005 1"/>
-        </equality>
-        <!-- Same logic as above... -->
-        <tendon>
-            <fixed name="${tf_prefix}lift_middle_mimic_higher">
-            <joint joint="${tf_prefix}ewellix_lift_lower_to_higher" coef="0.5"/>
-            <joint joint="${tf_prefix}middle_mimic_higher" coef="0.5"/>
-            </fixed>
-        </tendon>
-        <!-- The mimic joint is scaled by 50% in the URDF -->
-        <equality>
-            <joint name="${tf_prefix}upper_mimic_lower" joint1="${tf_prefix}ewellix_lift_lower_to_higher" joint2="${tf_prefix}middle_mimic_higher" polycoef="0 2 0 0 0"/>
-        </equality>
-        <sensor>
-            <force name="${tf_prefix}tcp_fts_sensor_force" site="${tf_prefix}ft_frame"/>
-            <torque name="${tf_prefix}tcp_fts_sensor_torque" site="${tf_prefix}ft_frame"/>
-        </sensor>
-        <!-- clr contacts -->
-        <contact>
-            <exclude body1="world" body2="${tf_prefix}vention_rail_carriage"/>
-            <exclude body1="world" body2="${tf_prefix}ewellix_lift_higher_link"/>
-            <exclude body1="world" body2="${tf_prefix}ewellix_lift_middle_link"/>
-            <exclude body1="${tf_prefix}vention_rail_carriage" body2="${tf_prefix}ewellix_lift_middle_link"/>
-        </contact>
-        <!-- environment contacts -->
+      </default>
+      <actuator>
+          <position joint="${tf_prefix}vention_rail_base_to_carriage" name="${tf_prefix}vention_rail_base_to_carriage" kp="25000" dampratio="1.0" ctrlrange="0.0 2.0" />
+          <position joint="${tf_prefix}ewellix_lift_lower_to_higher" name="${tf_prefix}ewellix_lift_lower_to_higher" kp="75000" dampratio="1.0" ctrlrange="0.0 0.7" />
+          <position class="clr_size4" name="${tf_prefix}shoulder_pan_joint" joint="${tf_prefix}shoulder_pan_joint"/>
+          <position class="clr_size4" name="${tf_prefix}shoulder_lift_joint" joint="${tf_prefix}shoulder_lift_joint"/>
+          <position class="clr_size3_limited" name="${tf_prefix}elbow_joint" joint="${tf_prefix}elbow_joint"/>
+          <position class="clr_size2" name="${tf_prefix}wrist_1_joint" joint="${tf_prefix}wrist_1_joint"/>
+          <position class="clr_size2" name="${tf_prefix}wrist_2_joint" joint="${tf_prefix}wrist_2_joint"/>
+          <position class="clr_size2" name="${tf_prefix}wrist_3_joint" joint="${tf_prefix}wrist_3_joint"/>
+          <position tendon="${tf_prefix}split" name="${tf_prefix}finger_1_joint" kp="10000" dampratio="3.0" ctrlrange="0.0 0.025" forcerange="-100 100"/>
+      </actuator>
+      <!--
+          This adds stability to the model by having a tendon that distributes the forces between both
+          joints, such that the equality constraint doesn't have to do that much work in order to equalize
+          both joints. Since both joints share the same sign, we split the force between both equally by
+          setting coef=0.5
+      -->
+      <tendon>
+          <fixed name="${tf_prefix}split">
+          <joint joint="${tf_prefix}finger_1_joint" coef="0.5"/>
+          <joint joint="${tf_prefix}finger_2_joint" coef="0.5"/>
+          </fixed>
+      </tendon>
+      <equality>
+          <joint joint1="${tf_prefix}finger_1_joint" joint2="${tf_prefix}finger_2_joint" polycoef="0 1 0 0 0" solimp="0.95 0.99 0.001" solref="0.005 1"/>
+      </equality>
+      <!-- Same logic as above... -->
+      <tendon>
+          <fixed name="${tf_prefix}lift_middle_mimic_higher">
+          <joint joint="${tf_prefix}ewellix_lift_lower_to_higher" coef="0.5"/>
+          <joint joint="${tf_prefix}middle_mimic_higher" coef="0.5"/>
+          </fixed>
+      </tendon>
+      <!-- The mimic joint is scaled by 50% in the URDF -->
+      <equality>
+          <joint name="${tf_prefix}upper_mimic_lower" joint1="${tf_prefix}ewellix_lift_lower_to_higher" joint2="${tf_prefix}middle_mimic_higher" polycoef="0 2 0 0 0"/>
+      </equality>
+      <sensor>
+          <force name="${tf_prefix}tcp_fts_sensor_force" site="${tf_prefix}ft_frame"/>
+          <torque name="${tf_prefix}tcp_fts_sensor_torque" site="${tf_prefix}ft_frame"/>
+      </sensor>
+      <!-- clr contacts -->
+      <contact>
+          <exclude body1="world" body2="${tf_prefix}vention_rail_carriage"/>
+          <exclude body1="world" body2="${tf_prefix}ewellix_lift_higher_link"/>
+          <exclude body1="world" body2="${tf_prefix}ewellix_lift_middle_link"/>
+          <exclude body1="${tf_prefix}vention_rail_carriage" body2="${tf_prefix}ewellix_lift_middle_link"/>
+      </contact>
+      <!-- environment contacts -->
+      <xacro:if value="${model_env}">
         <contact>
             <exclude body1="world" body2="lorge/hatch_face"/>
@@ -110,5 +114,29 @@
             <exclude body1="drawer_2_face" body2="recessed_latch_handle"/>
         </contact>
-    </raw_inputs>
+      </xacro:if>
+  </xacro:macro>
+  <!-- Can use `skip_tags` to include the macro in other files without duplicating inputs -->
+  <xacro:macro name="clr_mujoco_raw_inputs" params="
+    model_env:=true
+    tf_prefix:=''
+    defaults_prefix:=''
+    skip_tags:=false
+  ">
+    <xacro:unless value="${skip_tags}">
+      <raw_inputs>
+        <xacro:clr_mujoco_raw_inputs_content
+          model_env="${model_env}"
+          tf_prefix="${tf_prefix}"
+          defaults_prefix="${defaults_prefix}"
+        />
+      </raw_inputs>
+    </xacro:unless>
+    <xacro:if value="${skip_tags}">
+      <xacro:clr_mujoco_raw_inputs_content
+        model_env="${model_env}"
+        tf_prefix="${tf_prefix}"
+        defaults_prefix="${defaults_prefix}"
+      />
+    </xacro:if>
   </xacro:macro>
 </robot>

Commit message: Just move the tags to outside the macro

File: clr_mujoco_config/urdf/clr_mujoco_processed_inputs.xacro (robot description, xacro)
@@ -1,5 +1,5 @@
 <?xml version="1.0"?>
 <robot xmlns:xacro="http://wiki.ros.org/xacro">
-  <xacro:macro name="clr_mujoco_processed_inputs_content" params="
+  <xacro:macro name="clr_mujoco_processed_inputs" params="
     model_env:=true
     include_scene_objects:=false
@@ -43,27 +43,3 @@
       <modify_element type="joint" name="lorge/latch_spring" limited="true" springref="0.035" stiffness="10000" damping="2" armature="0.001"/>
   </xacro:macro>
-  <!-- Can use `skip_tags` to include the macro in other files without duplicating inputs -->
-  <xacro:macro name="clr_mujoco_processed_inputs" params="
-    model_env:=true
-    include_scene_objects:=false
-    tf_prefix:=''
-    skip_tags:=false
-  ">
-    <xacro:unless value="${skip_tags}">
-      <processed_inputs>
-        <xacro:clr_mujoco_processed_inputs_content
-          model_env="${model_env}"
-          include_scene_objects="${include_scene_objects}"
-          tf_prefix="${tf_prefix}"
-        />
-      </processed_inputs>
-    </xacro:unless>
-    <xacro:if value="${skip_tags}">
-      <xacro:clr_mujoco_processed_inputs_content
-        model_env="${model_env}"
-        include_scene_objects="${include_scene_objects}"
-        tf_prefix="${tf_prefix}"
-      />
-    </xacro:if>
-  </xacro:macro>
 </robot>

File: clr_mujoco_config/urdf/clr_mujoco_raw_inputs.xacro (robot description, xacro)
@@ -1,5 +1,5 @@
 <?xml version="1.0"?>
 <robot xmlns:xacro="http://wiki.ros.org/xacro">
-  <xacro:macro name="clr_mujoco_raw_inputs_content" params="
+  <xacro:macro name="clr_mujoco_raw_inputs" params="
     model_env:=true
     tf_prefix:=''
@@ -116,27 +116,3 @@
       </xacro:if>
   </xacro:macro>
-  <!-- Can use `skip_tags` to include the macro in other files without duplicating inputs -->
-  <xacro:macro name="clr_mujoco_raw_inputs" params="
-    model_env:=true
-    tf_prefix:=''
-    defaults_prefix:=''
-    skip_tags:=false
-  ">
-    <xacro:unless value="${skip_tags}">
-      <raw_inputs>
-        <xacro:clr_mujoco_raw_inputs_content
-          model_env="${model_env}"
-          tf_prefix="${tf_prefix}"
-          defaults_prefix="${defaults_prefix}"
-        />
-      </raw_inputs>
-    </xacro:unless>
-    <xacro:if value="${skip_tags}">
-      <xacro:clr_mujoco_raw_inputs_content
-        model_env="${model_env}"
-        tf_prefix="${tf_prefix}"
-        defaults_prefix="${defaults_prefix}"
-      />
-    </xacro:if>
-  </xacro:macro>
 </robot>
