Commit message: spacing issues

File: clr_mujoco_config/urdf/clr_mujoco_raw_inputs.xacro (robot description, xacro)
@@ -55,8 +55,8 @@
       -->
       <tendon>
-          <fixed name="${tf_prefix}split">
+        <fixed name="${tf_prefix}split">
           <joint joint="${tf_prefix}finger_1_joint" coef="0.5"/>
           <joint joint="${tf_prefix}finger_2_joint" coef="0.5"/>
-          </fixed>
+        </fixed>
       </tendon>
       <equality>
@@ -66,6 +66,6 @@
       <tendon>
           <fixed name="${tf_prefix}lift_middle_mimic_higher">
-          <joint joint="${tf_prefix}ewellix_lift_lower_to_higher" coef="0.5"/>
-          <joint joint="${tf_prefix}middle_mimic_higher" coef="0.5"/>
+            <joint joint="${tf_prefix}ewellix_lift_lower_to_higher" coef="0.5"/>
+            <joint joint="${tf_prefix}middle_mimic_higher" coef="0.5"/>
           </fixed>
       </tendon>
