Commit message: successfully switched controllers in sim

File: clr_mujoco_config/urdf/clr_mujoco_ros2_control_macros.xacro (robot description, xacro)
@@ -1,4 +1,5 @@
 <?xml version="1.0"?>
 <robot name="clr_mujoco_ros2_control_macros" xmlns:xacro="http://ros.org/wiki/xacro">
+  <xacro:include filename="$(find ur_description)/urdf/inc/ur_joint_control.xacro"/>
   <xacro:macro name="clr_mujoco_ros2_control_sensors" params="
     tf_prefix:=''
@@ -50,52 +51,9 @@
       <state_interface name="effort"/>
     </joint>
-    <joint name="${tf_prefix}shoulder_pan_joint">
-      <command_interface name="position"/>
-      <state_interface name="position">
-        <param name="initial_value">${3.1927}</param>
-      </state_interface>
-      <state_interface name="velocity"/>
-      <state_interface name="effort"/>
-    </joint>
-    <joint name="${tf_prefix}shoulder_lift_joint">
-      <command_interface name="position"/>
-      <state_interface name="position">
-        <param name="initial_value">${-2.3913}</param>
-      </state_interface>
-      <state_interface name="velocity"/>
-      <state_interface name="effort"/>
-    </joint>
-    <joint name="${tf_prefix}elbow_joint">
-      <command_interface name="position"/>
-      <state_interface name="position">
-        <param name="initial_value">${-1.7760}</param>
-      </state_interface>
-      <state_interface name="velocity"/>
-      <state_interface name="effort"/>
-    </joint>
-    <joint name="${tf_prefix}wrist_1_joint">
-      <command_interface name="position"/>
-      <state_interface name="position">
-        <param name="initial_value">${-0.4700}</param>
-      </state_interface>
-      <state_interface name="velocity"/>
-      <state_interface name="effort"/>
-    </joint>
-    <joint name="${tf_prefix}wrist_2_joint">
-      <command_interface name="position"/>
-      <state_interface name="position">
-        <param name="initial_value">${-1.6177}</param>
-      </state_interface>
-      <state_interface name="velocity"/>
-      <state_interface name="effort"/>
-    </joint>
-    <joint name="${tf_prefix}wrist_3_joint">
-      <command_interface name="position"/>
-      <state_interface name="position">
-        <param name="initial_value">${-1.6177}</param>
-      </state_interface>
-      <state_interface name="velocity"/>
-      <state_interface name="effort"/>
-    </joint>
+    <!-- UR joints -->
+    <xacro:ur_joint_control_description
+        tf_prefix="${tf_prefix}"
+        initial_positions="${dict(shoulder_pan_joint=3.1927,shoulder_lift_joint=-2.3913,elbow_joint=-1.7760,wrist_1_joint=-0.4700,wrist_2_joint=-1.6177,wrist_3_joint=-1.6177)}"
+      />
     <!-- Robotiq gripper -->
     <joint name="${tf_prefix}finger_1_joint">
