Commit message: fix previous result of merge conflict that got rid of effort control in sim

File: clr_mujoco_config/urdf/clr_mujoco_ros2_control_macros.xacro (robot description, xacro)
@@ -19,10 +19,9 @@
   <xacro:macro name="clr_mujoco_ros2_control_joints" params="
     tf_prefix:=''
-    initial_positions:=${dict()}
   ">
     <joint name="${tf_prefix}vention_rail_base_to_carriage">
       <command_interface name="position"/>
       <state_interface name="position">
-        <param name="initial_value">${initial_positions.get('vention_rail_base_to_carriage', 0.0)}</param>
+        <param name="initial_value">0.0</param>
       </state_interface>
       <state_interface name="velocity"/>
@@ -32,63 +31,20 @@
       <command_interface name="position"/>
       <state_interface name="position">
-        <!-- There's an issue where this can drop below 0 due to gravity so the default values starts it a little higher for now... -->
-        <param name="initial_value">${initial_positions.get('ewellix_lift_lower_to_higher', 0.01)}</param>
+        <!-- There's an issue where this can drop below 0 due to gravity so starting it a little higher for now... -->
+        <param name="initial_value">0.01</param>
       </state_interface>
       <state_interface name="velocity"/>
       <state_interface name="effort"/>
     </joint>
-    <joint name="${tf_prefix}shoulder_pan_joint">
-      <command_interface name="position"/>
-      <state_interface name="position">
-        <param name="initial_value">${initial_positions.get('shoulder_pan_joint', 3.1927)}</param>
-      </state_interface>
-      <state_interface name="velocity"/>
-      <state_interface name="effort"/>
-    </joint>
-    <joint name="${tf_prefix}shoulder_lift_joint">
-      <command_interface name="position"/>
-      <state_interface name="position">
-        <param name="initial_value">${initial_positions.get('shoulder_lift_joint', -2.3913)}</param>
-      </state_interface>
-      <state_interface name="velocity"/>
-      <state_interface name="effort"/>
-    </joint>
-    <joint name="${tf_prefix}elbow_joint">
-      <command_interface name="position"/>
-      <state_interface name="position">
-        <param name="initial_value">${initial_positions.get('elbow_joint', -1.7760)}</param>
-      </state_interface>
-      <state_interface name="velocity"/>
-      <state_interface name="effort"/>
-    </joint>
-    <joint name="${tf_prefix}wrist_1_joint">
-      <command_interface name="position"/>
-      <state_interface name="position">
-        <param name="initial_value">${initial_positions.get('wrist_1_joint', -0.4700)}</param>
-      </state_interface>
-      <state_interface name="velocity"/>
-      <state_interface name="effort"/>
-    </joint>
-    <joint name="${tf_prefix}wrist_2_joint">
-      <command_interface name="position"/>
-      <state_interface name="position">
-        <param name="initial_value">${initial_positions.get('wrist_2_joint', -1.6177)}</param>
-      </state_interface>
-      <state_interface name="velocity"/>
-      <state_interface name="effort"/>
-    </joint>
-    <joint name="${tf_prefix}wrist_3_joint">
-      <command_interface name="position"/>
-      <state_interface name="position">
-        <param name="initial_value">${initial_positions.get('wrist_3_joint', -1.6177)}</param>
-      </state_interface>
-      <state_interface name="velocity"/>
-      <state_interface name="effort"/>
-    </joint>
+    <!-- UR joints -->
+    <xacro:ur_joint_control_description
+        tf_prefix="${tf_prefix}"
+        initial_positions="${dict(shoulder_pan_joint=3.1927,shoulder_lift_joint=-2.3913,elbow_joint=-1.7760,wrist_1_joint=-0.4700,wrist_2_joint=-1.6177,wrist_3_joint=-1.6177)}"
+      />
     <!-- Robotiq gripper -->
     <joint name="${tf_prefix}finger_1_joint">
       <command_interface name="position"/>
       <state_interface name="position">
-        <param name="initial_value">${initial_positions.get('finger_1_joint', 0.025)}</param>
+        <param name="initial_value">0.025</param>
       </state_interface>
       <state_interface name="velocity"/>

Commit message: Revert "fix previous result of merge conflict that got rid of effort control in sim"
This reverts commit a9f8ea288da68f011ebd0980ccf0850cce50f8c8.

File: clr_mujoco_config/urdf/clr_mujoco_ros2_control_macros.xacro (robot description, xacro)
@@ -19,9 +19,10 @@
   <xacro:macro name="clr_mujoco_ros2_control_joints" params="
     tf_prefix:=''
+    initial_positions:=${dict()}
   ">
     <joint name="${tf_prefix}vention_rail_base_to_carriage">
       <command_interface name="position"/>
       <state_interface name="position">
-        <param name="initial_value">0.0</param>
+        <param name="initial_value">${initial_positions.get('vention_rail_base_to_carriage', 0.0)}</param>
       </state_interface>
       <state_interface name="velocity"/>
@@ -31,20 +32,63 @@
       <command_interface name="position"/>
       <state_interface name="position">
-        <!-- There's an issue where this can drop below 0 due to gravity so starting it a little higher for now... -->
-        <param name="initial_value">0.01</param>
+        <!-- There's an issue where this can drop below 0 due to gravity so the default values starts it a little higher for now... -->
+        <param name="initial_value">${initial_positions.get('ewellix_lift_lower_to_higher', 0.01)}</param>
       </state_interface>
       <state_interface name="velocity"/>
       <state_interface name="effort"/>
     </joint>
-    <!-- UR joints -->
-    <xacro:ur_joint_control_description
-        tf_prefix="${tf_prefix}"
-        initial_positions="${dict(shoulder_pan_joint=3.1927,shoulder_lift_joint=-2.3913,elbow_joint=-1.7760,wrist_1_joint=-0.4700,wrist_2_joint=-1.6177,wrist_3_joint=-1.6177)}"
-      />
+    <joint name="${tf_prefix}shoulder_pan_joint">
+      <command_interface name="position"/>
+      <state_interface name="position">
+        <param name="initial_value">${initial_positions.get('shoulder_pan_joint', 3.1927)}</param>
+      </state_interface>
+      <state_interface name="velocity"/>
+      <state_interface name="effort"/>
+    </joint>
+    <joint name="${tf_prefix}shoulder_lift_joint">
+      <command_interface name="position"/>
+      <state_interface name="position">
+        <param name="initial_value">${initial_positions.get('shoulder_lift_joint', -2.3913)}</param>
+      </state_interface>
+      <state_interface name="velocity"/>
+      <state_interface name="effort"/>
+    </joint>
+    <joint name="${tf_prefix}elbow_joint">
+      <command_interface name="position"/>
+      <state_interface name="position">
+        <param name="initial_value">${initial_positions.get('elbow_joint', -1.7760)}</param>
+      </state_interface>
+      <state_interface name="velocity"/>
+      <state_interface name="effort"/>
+    </joint>
+    <joint name="${tf_prefix}wrist_1_joint">
+      <command_interface name="position"/>
+      <state_interface name="position">
+        <param name="initial_value">${initial_positions.get('wrist_1_joint', -0.4700)}</param>
+      </state_interface>
+      <state_interface name="velocity"/>
+      <state_interface name="effort"/>
+    </joint>
+    <joint name="${tf_prefix}wrist_2_joint">
+      <command_interface name="position"/>
+      <state_interface name="position">
+        <param name="initial_value">${initial_positions.get('wrist_2_joint', -1.6177)}</param>
+      </state_interface>
+      <state_interface name="velocity"/>
+      <state_interface name="effort"/>
+    </joint>
+    <joint name="${tf_prefix}wrist_3_joint">
+      <command_interface name="position"/>
+      <state_interface name="position">
+        <param name="initial_value">${initial_positions.get('wrist_3_joint', -1.6177)}</param>
+      </state_interface>
+      <state_interface name="velocity"/>
+      <state_interface name="effort"/>
+    </joint>
     <!-- Robotiq gripper -->
     <joint name="${tf_prefix}finger_1_joint">
       <command_interface name="position"/>
       <state_interface name="position">
-        <param name="initial_value">0.025</param>
+        <param name="initial_value">${initial_positions.get('finger_1_joint', 0.025)}</param>
       </state_interface>
       <state_interface name="velocity"/>

Commit message: fix lorge/latch_spring

File: clr_mujoco_config/urdf/clr_mujoco_ros2_control_macros.xacro (robot description, xacro)
@@ -125,7 +125,4 @@
       <state_interface name="position"/>
     </joint>
-    <joint name="lorge/latch_spring">
-      <state_interface name="position"/>
-    </joint>
     <joint name="lorge/external_rotary_joint">
       <state_interface name="position"/>
